Commit message: fix: namespace correction

File: src/ur3e_hande_robot_description/urdf/robotiq_hande.urdf.xacro (robot description, xacro)
@@ -11,5 +11,5 @@
         <origin xyz="0 0 0" rpy="0 0 0" />
         <geometry>
-          <mesh filename="package://ur3e_hande_description/meshes/hande/visual/hand-e.dae" scale="0.001 0.001 0.001"/>
+          <mesh filename="package://ur3e_hande_robot_description/meshes/hande/visual/hand-e.dae" scale="0.001 0.001 0.001"/>
         </geometry>
         <material name="Gazebo/Black">
@@ -20,5 +20,5 @@
         <origin xyz="0 0 0" rpy="0 0 0" />
         <geometry>
-          <mesh filename="package://ur3e_hande_description/meshes/hande/collision/hand-e.stl" scale="0.001 0.001 0.001"/>
+          <mesh filename="package://ur3e_hande_robot_description/meshes/hande/collision/hand-e.stl" scale="0.001 0.001 0.001"/>
         </geometry>
       </collision>
@@ -37,5 +37,5 @@
         <origin rpy="0 0 0" xyz="0 0 0"/>
         <geometry>
-          <mesh filename="package://ur3e_hande_description/meshes/hande/visual/finger_1.dae" scale="0.001 0.001 0.001"/>
+          <mesh filename="package://ur3e_hande_robot_description/meshes/hande/visual/finger_1.dae" scale="0.001 0.001 0.001"/>
         </geometry>
         <material name="Gazebo/Grey">
@@ -46,5 +46,5 @@
         <origin rpy="0 0 0" xyz="0 0 0"/>
         <geometry>
-          <mesh filename="package://ur3e_hande_description/meshes/hande/collision/finger_1.stl" scale="0.001 0.001 0.001"/>
+          <mesh filename="package://ur3e_hande_robot_description/meshes/hande/collision/finger_1.stl" scale="0.001 0.001 0.001"/>
         </geometry>
       </collision>
@@ -63,5 +63,5 @@
         <origin rpy="0 0 0" xyz="0 0 0"/>
         <geometry>
-          <mesh filename="package://ur3e_hande_description/meshes/hande/vision/finger_2.dae" scale="0.001 0.001 0.001"/>
+          <mesh filename="package://ur3e_hande_robot_description/meshes/hande/vision/finger_2.dae" scale="0.001 0.001 0.001"/>
         </geometry>
         <material name="Gazebo/Grey">
@@ -72,5 +72,5 @@
         <origin rpy="0 0 0" xyz="0 0 0"/>
         <geometry>
-          <mesh filename="package://ur3e_hande_description/meshes/hande/collision/finger_2.stl" scale="0.001 0.001 0.001"/>
+          <mesh filename="package://ur3e_hande_robot_description/meshes/hande/collision/finger_2.stl" scale="0.001 0.001 0.001"/>
         </geometry>
       </collision>

File: src/ur3e_hande_robot_description/urdf/ur.urdf.xacro (robot description, xacro)
@@ -4,5 +4,5 @@
    <xacro:arg name="name" default="ur"/>
    <!-- import main macro -->
-   <xacro:include filename="$(find ur3e_hande_duplicate_description)/urdf/ur_macro.xacro"/>
+   <xacro:include filename="$(find ur3e_hande_robot_description)/urdf/ur_macro.xacro"/>
    <!-- possible 'ur_type' values: ur3, ur3e, ur5, ur5e, ur10, ur10e, ur16e -->
    <!-- the default value should raise an error in case this was called without defining the type -->
@@ -10,8 +10,8 @@
    <!-- parameters -->
    <xacro:arg name="prefix" default="" />
-   <xacro:arg name="joint_limit_params" default="$(find ur3e_hande_duplicate_description)/config/$(arg ur_type)/joint_limits.yaml"/>
-   <xacro:arg name="kinematics_params" default="$(find ur3e_hande_duplicate_description)/config/$(arg ur_type)/default_kinematics.yaml"/>
-   <xacro:arg name="physical_params" default="$(find ur3e_hande_duplicate_description)/config/$(arg ur_type)/physical_parameters.yaml"/>
-   <xacro:arg name="visual_params" default="$(find ur3e_hande_duplicate_description)/config/$(arg ur_type)/visual_parameters.yaml"/>
+   <xacro:arg name="joint_limit_params" default="$(find ur3e_hande_robot_description)/config/$(arg ur_type)/joint_limits.yaml"/>
+   <xacro:arg name="kinematics_params" default="$(find ur3e_hande_robot_description)/config/$(arg ur_type)/default_kinematics.yaml"/>
+   <xacro:arg name="physical_params" default="$(find ur3e_hande_robot_description)/config/$(arg ur_type)/physical_parameters.yaml"/>
+   <xacro:arg name="visual_params" default="$(find ur3e_hande_robot_description)/config/$(arg ur_type)/visual_parameters.yaml"/>
    <xacro:arg name="transmission_hw_interface" default=""/>
    <xacro:arg name="safety_limits" default="false"/>
@@ -43,5 +43,5 @@
    <xacro:arg name="simulation_controllers" default="" />
    <!-- initial position for simulations (Fake Hardware, Gazebo, Ignition) -->
-   <xacro:arg name="initial_positions_file" default="$(find ur3e_hande_duplicate_description)/config/initial_positions.yaml"/>
+   <xacro:arg name="initial_positions_file" default="$(find ur3e_hande_robot_description)/config/initial_positions.yaml"/>
    <!-- convert to property to use substitution in function -->
    <xacro:property name="initial_positions_file" default="$(arg initial_positions_file)"/>

File: src/ur3e_hande_robot_description/urdf/ur_macro.xacro (robot description, xacro)
@@ -42,6 +42,6 @@
      - Muhammad Asif Rana
   -->
-  <xacro:include filename="$(find ur3e_hande_duplicate_description)/urdf/inc/ur_transmissions.xacro" />
-  <xacro:include filename="$(find ur3e_hande_duplicate_description)/urdf/inc/ur_common.xacro" />
+  <xacro:include filename="$(find ur3e_hande_robot_description)/urdf/inc/ur_transmissions.xacro" />
+  <xacro:include filename="$(find ur3e_hande_robot_description)/urdf/inc/ur_common.xacro" />
   <xacro:macro name="ur_robot" params="
     name
@@ -88,5 +88,5 @@
       force_abs_paths="${sim_gazebo or sim_ignition}"/>
     <!-- ros2 control include -->
-    <xacro:include filename="$(find ur3e_hande_duplicate_description)/urdf/ur.ros2_control.xacro" />
+    <xacro:include filename="$(find ur3e_hande_robot_description)/urdf/ur.ros2_control.xacro" />
     <!-- ros2 control instance -->
     <xacro:ur_ros2_control
@@ -255,5 +255,5 @@
         <origin xyz="0 0 0" rpy="0 0 0" />
         <geometry>
-          <mesh filename="package://ur3e_hande_duplicate_description/meshes/hande/visual/hand-e.dae" scale="0.001 0.001 0.001" />
+          <mesh filename="package://ur3e_hande_robot_description/meshes/hande/visual/hand-e.dae" scale="0.001 0.001 0.001" />
         </geometry>
         <material name="Gazebo/Black">
@@ -264,5 +264,5 @@
         <origin xyz="0 0 0" rpy="0 0 0" />
         <geometry>
-          <mesh filename="package://ur3e_hande_duplicate_description/meshes/hande/collision/hand-e.stl" scale="0.001 0.001 0.001"/>
+          <mesh filename="package://ur3e_hande_robot_description/meshes/hande/collision/hand-e.stl" scale="0.001 0.001 0.001"/>
         </geometry>
       </collision>
@@ -280,5 +280,5 @@
         <origin rpy="0 0 0" xyz="0 0 0"/>
         <geometry>
-          <mesh filename="package://ur3e_hande_duplicate_description/meshes/hande/visual/finger_1.dae" scale="0.001 0.001 0.001"/>
+          <mesh filename="package://ur3e_hande_robot_description/meshes/hande/visual/finger_1.dae" scale="0.001 0.001 0.001"/>
         </geometry>
         <material name="Gazebo/Grey">
@@ -289,5 +289,5 @@
         <origin rpy="0 0 0" xyz="0 0 0"/>
         <geometry>
-          <mesh filename="package://ur3e_hande_duplicate_description/meshes/hande/collision/finger_1.stl" scale="0.001 0.001 0.001"/>
+          <mesh filename="package://ur3e_hande_robot_description/meshes/hande/collision/finger_1.stl" scale="0.001 0.001 0.001"/>
         </geometry>
       </collision>
@@ -305,5 +305,5 @@
         <origin rpy="0 0 0" xyz="0 0 0"/>
         <geometry>
-          <mesh filename="package://ur3e_hande_duplicate_description/meshes/hande/visual/finger_2.dae" scale="0.001 0.001 0.001"/>
+          <mesh filename="package://ur3e_hande_robot_description/meshes/hande/visual/finger_2.dae" scale="0.001 0.001 0.001"/>
         </geometry>
         <material name="Gazebo/Grey">
@@ -314,5 +314,5 @@
         <origin rpy="0 0 0" xyz="0 0 0"/>
         <geometry>
-          <mesh filename="package://ur3e_hande_duplicate_description/meshes/hande/collision/finger_2.stl" scale="0.001 0.001 0.001"/>
+          <mesh filename="package://ur3e_hande_robot_description/meshes/hande/collision/finger_2.stl" scale="0.001 0.001 0.001"/>
         </geometry>
       </collision>
