Commit message: fix: hande intermediate steps

File: src/ur3e_hande_robot_description/urdf/hande_extension.urdf.xacro (robot description, xacro)
@@ -2,5 +2,11 @@
 <robot xmlns:xacro="http://wiki.ros.org/xacro" name="$(arg name)">
   <xacro:include filename="$(find ur_description)/urdf/ur.urdf.xacro"/>
-  <xacro:macro name="read_model_data" params="joint_limits_parameters_file kinematics_parameters_file physical_parameters_file visual_parameters_file force_abs_paths">
+  <xacro:macro name="read_model_data_2" params="joint_limits_parameters_file kinematics_parameters_file physical_parameters_file visual_parameters_file force_abs_paths">
+     <xacro:read_model_data
+      joint_limits_parameters_file="${joint_limits_parameters_file}"
+      kinematics_parameters_file="${kinematics_parameters_file}"
+      physical_parameters_file="${physical_parameters_file}"
+      visual_parameters_file="${visual_parameters_file}"
+      force_abs_paths="${sim_gazebo or sim_ignition}"/>
     <xacro:property name="hande_base_mass" value="${sec_inertia_parameters['hande_base_mass']}" scope="parent"/>
     <xacro:property name="left_finger_mass" value="${sec_inertia_parameters['left_finger_mass']}" scope="parent"/>
@@ -19,260 +25,9 @@
     <xacro:property name="finger_radius" value="${sec_inertia_parameters['finger_radius']}" scope="parent"/>
 </xacro:macro>
- <xacro:macro name="ur_ros2_control" params="
-    name
-    prefix
-    use_fake_hardware:=false fake_sensor_commands:=false
-    sim_gazebo:=false
-    sim_ignition:=false
-    headless_mode:=false
-    initial_positions:=${dict(shoulder_pan_joint=0.0,shoulder_lift_joint=-1.57,elbow_joint=0.0,wrist_1_joint=-1.57,wrist_2_joint=0.0,wrist_3_joint=0.0,joint_finger=0.01,robotiq_hande_base_to_right_finger=0.01)}
-    use_tool_communication:=false
-    script_filename output_recipe_filename
-    input_recipe_filename tf_prefix
-    hash_kinematics robot_ip
-    tool_voltage:=0 tool_parity:=0 tool_baud_rate:=115200 tool_stop_bits:=1
-    tool_rx_idle_chars:=1.5 tool_tx_idle_chars:=3.5 tool_device_name:=/tmp/ttyUR tool_tcp_port:=54321
-    reverse_port:=50001
-    script_sender_port:=50002
-    reverse_ip:=0.0.0.0
-    script_command_port:=50004">
-    <ros2_control name="${name}" type="system">
-      <!-- custom changes for hande -->
-      <joint name="${prefix}joint_finger">
-        <command_interface name="position">
-          <param name="min">-0.1</param>
-          <param name="max">0.1</param>
-        </command_interface>
-        <command_interface name="velocity">
-          <param name="min">-0.025</param>
-          <param name="max">0.025</param>
-        </command_interface>
-        <state_interface name="position">
-          <!-- initial position for the FakeSystem and simulation -->
-          <param name="initial_value">${initial_positions['joint_finger']}</param>
-        </state_interface>
-        <state_interface name="velocity"/>
-        <state_interface name="effort"/>
-      </joint>
-      <joint name="robotiq_hande_base_to_${prefix}right_finger">
-        <command_interface name="position">
-          <param name="min">-0.1</param>
-          <param name="max">0.1</param>
-        </command_interface>
-        <command_interface name="velocity">
-          <param name="min">-0.025</param>
-          <param name="max">0.025</param>
-        </command_interface>
-        <state_interface name="position">
-          <!-- initial position for the FakeSystem and simulation -->
-          <param name="initial_value">${initial_positions['joint_finger']}</param>
-        </state_interface>
-        <state_interface name="velocity"/>
-        <state_interface name="effort"/>
-      </joint>
-  </ros2_control>
-  </xacro:macro>
-<xacro:macro name="ur_robot">
-   <xacro:ur_robot
-     name="$(arg name)"
-     tf_prefix="$(arg tf_prefix)"
-     parent="world"
-     joint_limits_parameters_file="$(arg joint_limit_params)"
-     kinematics_parameters_file="$(arg kinematics_params)"
-     physical_parameters_file="$(arg physical_params)"
-     visual_parameters_file="$(arg visual_params)"
-     transmission_hw_interface="$(arg transmission_hw_interface)"
-     safety_limits="$(arg safety_limits)"
-     safety_pos_margin="$(arg safety_pos_margin)"
-     safety_k_position="$(arg safety_k_position)"
-     use_fake_hardware="$(arg use_fake_hardware)"
-     fake_sensor_commands="$(arg fake_sensor_commands)"
-     sim_gazebo="$(arg sim_gazebo)"
-     sim_ignition="$(arg sim_ignition)"
-     headless_mode="$(arg headless_mode)"
-     initial_positions="${xacro.load_yaml(initial_positions_file)}"
-     use_tool_communication="$(arg use_tool_communication)"
-     tool_voltage="$(arg tool_voltage)"
-     tool_parity="$(arg tool_parity)"
-     tool_baud_rate="$(arg tool_baud_rate)"
-     tool_stop_bits="$(arg tool_stop_bits)"
-     tool_rx_idle_chars="$(arg tool_rx_idle_chars)"
-     tool_tx_idle_chars="$(arg tool_tx_idle_chars)"
-     tool_device_name="$(arg tool_device_name)"
-     tool_tcp_port="$(arg tool_tcp_port)"
-     robot_ip="$(arg robot_ip)"
-     script_filename="$(arg script_filename)"
-     output_recipe_filename="$(arg output_recipe_filename)"
-     input_recipe_filename="$(arg input_recipe_filename)"
-     reverse_ip="$(arg reverse_ip)"
-     script_command_port="$(arg script_command_port)"
-     reverse_port="$(arg reverse_port)"
-     script_sender_port="$(arg script_sender_port)"
-     trajectory_port="$(arg trajectory_port)"
-     >
-     <origin xyz="0 0 0" rpy="0 0 0" />          <!-- position robot in the world -->
-   </xacro:ur_robot>
-    <!-- customization to include hande -->
-    <link name="${prefix}robotiq_hande_base_link">
-<!--       <inertial>
-        <origin xyz="0 0 0.04607" rpy="0 0 0" />
-        <mass value="0.86387" />
-        <inertia ixx="1017560E-9" ixy="0" ixz="2235E-9" iyy="1028041E-9" iyz="0" izz="489810E-9" />
-      </inertial> -->
-      <visual>
-        <origin xyz="0 0 0" rpy="0 0 0" />
-        <geometry>
-          <mesh filename="package://ur3e_hande_robot_description/meshes/hande/visual/hand-e.dae" scale="0.001 0.001 0.001" />
-        </geometry>
-        <material name="Gazebo/Black">
-          <color rgba="0.1 0.1 0.1 1" />
-        </material>
-      </visual>
-      <collision>
-        <origin xyz="0 0 0" rpy="0 0 0" />
-        <geometry>
-          <mesh filename="package://ur3e_hande_robot_description/meshes/hande/collision/hand-e.stl" scale="0.001 0.001 0.001"/>
-        </geometry>
-      </collision>
-      <xacro:cylinder_inertial radius="${hande_base_inertia_radius}" length="${hande_base_inertia_length}"  mass="${hande_base_mass}">
-        <origin xyz="0.0 0.0 ${-0.5 * hande_base_inertia_length}" rpy="0 0 0" />
-      </xacro:cylinder_inertial>
-    </link>
-    <link name="${prefix}left_finger">
-<!--       <inertial>
-        <origin rpy="0 0 0" xyz="0.02262 -0.00759 0.00738"/>
-        <mass value="0.03804"/>
-        <inertia ixx="13567E-9" ixy="1849E-9" ixz="3622E-9" iyy="15784E-9" iyz="3616E-9" izz="7478E-9"/>
-      </inertial> -->
-      <visual>
-        <origin rpy="0 0 0" xyz="0 0 0"/>
-        <geometry>
-          <mesh filename="package://ur3e_hande_robot_description/meshes/hande/visual/finger_1.dae" scale="0.001 0.001 0.001"/>
-        </geometry>
-        <material name="Gazebo/Grey">
-          <color rgba="0.1 0.1 0.1 1"/>
-        </material>
-      </visual>
-      <collision>
-        <origin rpy="0 0 0" xyz="0 0 0"/>
-        <geometry>
-          <mesh filename="package://ur3e_hande_robot_description/meshes/hande/collision/finger_1.stl" scale="0.001 0.001 0.001"/>
-        </geometry>
-      </collision>
-      <xacro:cylinder_inertial radius="${left_finger_inertia_radius}" length="${left_finger_inertia_length}"  mass="${left_finger_mass}">
-        <origin xyz="0.0 0.0 ${-0.5 * left_finger_inertia_length}" rpy="0 0 0" />
-      </xacro:cylinder_inertial>
-    </link>
-    <link name="${prefix}right_finger">
-<!--       <inertial>
-        <origin rpy="0 0 0" xyz="-0.02262 0.00759 0.00738"/>
-        <mass value="0.03804"/>
-        <inertia ixx="13567E-9" ixy="1849E-9" ixz="-3622E-9" iyy="15784E-9" iyz="-3616E-9" izz="7478E-9"/>
-      </inertial> -->
-      <visual>
-        <origin rpy="0 0 0" xyz="0 0 0"/>
-        <geometry>
-          <mesh filename="package://ur3e_hande_robot_description/meshes/hande/visual/finger_2.dae" scale="0.001 0.001 0.001"/>
-        </geometry>
-        <material name="Gazebo/Grey">
-          <color rgba="0.1 0.1 0.1 1"/>
-        </material>
-      </visual>
-      <collision>
-        <origin rpy="0 0 0" xyz="0 0 0"/>
-        <geometry>
-          <mesh filename="package://ur3e_hande_robot_description/meshes/hande/collision/finger_2.stl" scale="0.001 0.001 0.001"/>
-        </geometry>
-      </collision>
-      <xacro:cylinder_inertial radius="${right_finger_inertia_radius}" length="${right_finger_inertia_length}"  mass="${right_finger_mass}">
-        <origin xyz="0.0 0.0 ${-0.5 * right_finger_inertia_length}" rpy="0 0 0" />
-      </xacro:cylinder_inertial>
-    </link>
-    <!-- hande installation -->
-    <joint name="${prefix}joint_finger" type="prismatic">
-      <origin rpy="0 0 0" xyz="0 0 0.099"/>
-      <parent link="${prefix}robotiq_hande_base_link"/>
-      <child link="${prefix}left_finger"/>
-      <axis xyz="-1 0 0"/>
-      <limit effort="130" lower="0" upper="0.025" velocity="0.15"/>
-    </joint>
-    <joint name="robotiq_hande_base_to_${prefix}right_finger" type="prismatic">
-      <origin rpy="0 0 0" xyz="0 0 0.099"/>
-      <parent link="${prefix}robotiq_hande_base_link"/>
-      <child link="${prefix}right_finger"/>
-      <axis xyz="1 0 0"/>
-      <limit effort="130" lower="0" upper="0.025" velocity="0.15"/>
-      <mimic joint="${prefix}joint_finger" multiplier="1" offset="0"/>
-    </joint>
-<!--     <link name="${prefix}ft_frame"/>
-    <joint name="${prefix}wrist_3_link-ft_frame" type="fixed">
-      <parent link="${prefix}wrist_3_link"/>
-      <child link="${prefix}ft_frame"/>
-      <origin xyz="0 0 0" rpy="${pi} 0 0"/>
-    </joint> -->
-    <!-- ROS-Industrial 'base' frame - base_link to UR 'Base' Coordinates transform -->
-    <link name="${prefix}base"/>
-    <joint name="${prefix}base_link-base_fixed_joint" type="fixed">
-      <!-- Note the rotation over Z of pi radians - as base_link is REP-103
-           aligned (i.e., has X+ forward, Y+ left and Z+ up), this is needed
-           to correctly align 'base' with the 'Base' coordinate system of
-           the UR controller.
-      -->
-      <origin xyz="0 0 0" rpy="0 0 ${pi}"/>
-      <parent link="${prefix}base_link"/>
-      <child link="${prefix}base"/>
-    </joint>
-    <!-- ROS-Industrial 'flange' frame - attachment point for EEF models -->
-    <!-- <link name="${prefix}flange" />
-    <joint name="${prefix}wrist_3-flange" type="fixed">
-      <parent link="${prefix}wrist_3_link" />
-      <child link="${prefix}flange" />
-      <origin xyz="0 0 0" rpy="0 ${-pi/2.0} ${-pi/2.0}" />
-    </joint> -->
-    <joint name="${prefix}hande_to_wrist_flange" type="fixed">
-      <parent link="${prefix}tool0" />
-      <child link="${prefix}robotiq_hande_base_link" />
-      <origin xyz="0 0 0" rpy="0 0 0" />
-    </joint>
-</xacro:macro>
-   <!-- arm -->
-   <xacro:ur_robot
-     name="$(arg name)"
-     tf_prefix="$(arg tf_prefix)"
-     parent="world"
-     joint_limits_parameters_file="$(arg joint_limit_params)"
-     kinematics_parameters_file="$(arg kinematics_params)"
-     physical_parameters_file="$(arg physical_params)"
-     visual_parameters_file="$(arg visual_params)"
-     transmission_hw_interface="$(arg transmission_hw_interface)"
-     safety_limits="$(arg safety_limits)"
-     safety_pos_margin="$(arg safety_pos_margin)"
-     safety_k_position="$(arg safety_k_position)"
-     use_fake_hardware="$(arg use_fake_hardware)"
-     fake_sensor_commands="$(arg fake_sensor_commands)"
-     sim_gazebo="$(arg sim_gazebo)"
-     sim_ignition="$(arg sim_ignition)"
-     headless_mode="$(arg headless_mode)"
-     initial_positions="${xacro.load_yaml(initial_positions_file)}"
-     use_tool_communication="$(arg use_tool_communication)"
-     tool_voltage="$(arg tool_voltage)"
-     tool_parity="$(arg tool_parity)"
-     tool_baud_rate="$(arg tool_baud_rate)"
-     tool_stop_bits="$(arg tool_stop_bits)"
-     tool_rx_idle_chars="$(arg tool_rx_idle_chars)"
-     tool_tx_idle_chars="$(arg tool_tx_idle_chars)"
-     tool_device_name="$(arg tool_device_name)"
-     tool_tcp_port="$(arg tool_tcp_port)"
-     robot_ip="$(arg robot_ip)"
-     script_filename="$(arg script_filename)"
-     output_recipe_filename="$(arg output_recipe_filename)"
-     input_recipe_filename="$(arg input_recipe_filename)"
-     reverse_ip="$(arg reverse_ip)"
-     script_command_port="$(arg script_command_port)"
-     reverse_port="$(arg reverse_port)"
-     script_sender_port="$(arg script_sender_port)"
-     trajectory_port="$(arg trajectory_port)"
-     >
-     <origin xyz="0 0 0" rpy="0 0 0" />          <!-- position robot in the world -->
-   </xacro:ur_robot>
+    <xacro:read_model_data_2
+      joint_limits_parameters_file="${joint_limits_parameters_file}"
+      kinematics_parameters_file="${kinematics_parameters_file}"
+      physical_parameters_file="${physical_parameters_file}"
+      visual_parameters_file="${visual_parameters_file}"
+      force_abs_paths="${sim_gazebo or sim_ignition}"/>
 </robot>

Commit message: fix: debug xacro

File: src/ur3e_hande_robot_description/urdf/hande_extension.urdf.xacro (robot description, xacro)
@@ -1,6 +1,10 @@
 <?xml version="1.0"?>
 <robot xmlns:xacro="http://wiki.ros.org/xacro" name="$(arg name)">
-  <xacro:include filename="$(find ur_description)/urdf/ur_macro.xacro"/>
-  <!-- <xacro:include filename="$(find ur3e_hande_robot_description)/urdf/hande.xacro"/> -->
+   <!-- robot name parameter -->
+   <xacro:arg name="name" default="ur"/>
+   <!-- import main macro -->
+   <xacro:include filename="$(find ur3e_hande_robot_description)/urdf/ur_macro.xacro"/>
+   <!-- possible 'ur_type' values: ur3, ur3e, ur5, ur5e, ur10, ur10e, ur16e -->
+   <!-- the default value should raise an error in case this was called without defining the type -->
    <xacro:arg name="ur_type" default="ur5x"/>
    <!-- parameters -->
@@ -32,8 +36,4 @@
    <xacro:arg name="tool_device_name" default="/tmp/ttyUR" />
    <xacro:arg name="tool_tcp_port" default="54321" />
-  <xacro:arg name="hande_joint_limit_params" default="$(find ur3e_hande_robot_description)/config/hande/joint_limits.yaml"/>
-  <xacro:arg name="hande_kinematics_params" default="$(find ur3e_hande_robot_description)/config/hande/default_kinematics.yaml"/>
-  <xacro:arg name="hande_physical_params" default="$(find ur3e_hande_robot_description)/config/hande/physical_parameters.yaml"/>
-  <xacro:arg name="hande_visual_params" default="$(find ur3e_hande_robot_description)/config/hande/visual_parameters.yaml"/>
      <!-- Simulation parameters -->
    <xacro:arg name="use_fake_hardware" default="false" />
@@ -42,25 +42,11 @@
    <xacro:arg name="sim_ignition" default="false" />
    <xacro:arg name="simulation_controllers" default="" />
-    <!-- <xacro:robotiq_hande
-     name="$(arg name)"
-     prefix="$(arg prefix)"
-     parent="world"
-     joint_limits_parameters_file="$(arg hande_joint_limit_params)"
-     kinematics_parameters_file="$(arg hande_kinematics_params)"
-     physical_parameters_file="$(arg hande_physical_params)"
-     visual_parameters_file="$(arg hande_visual_params)"
-   /> -->
-    <!-- name
-    prefix
-    parent
-    *origin
-    joint_limits_parameters_file
-    kinematics_parameters_file
-    physical_parameters_file
-    visual_parameters_file
-    initial_positions:=${dict(joint_finger=0.01,robotiq_hande_base_to_right_finger=0.01)}" >
-  -->
+   <!-- initial position for simulations (Fake Hardware, Gazebo, Ignition) -->
+   <xacro:arg name="initial_positions_file" default="$(find ur3e_hande_robot_description)/config/initial_positions.yaml"/>
+   <!-- convert to property to use substitution in function -->
+   <xacro:property name="initial_positions_file" default="$(arg initial_positions_file)"/>
    <!-- create link fixed to the "world" -->
    <link name="world" />
+   <!-- arm -->
    <xacro:ur_robot
      name="$(arg name)"
@@ -97,17 +83,26 @@
      script_command_port="$(arg script_command_port)"
      >
-<!--
-    <joint name="${prefix}hande_to_wrist_flange" type="fixed">
-      <parent link="${prefix}flange" />
-      <child link="${prefix}robotiq_hande_base_link" />
-      <origin xyz="0 0 0" rpy="0 0 0" />
-    </joint> -->
      <origin xyz="0 0 0" rpy="0 0 0" />          <!-- position robot in the world -->
    </xacro:ur_robot>
-    <!-- <xacro:read_model_data
-      joint_limits_parameters_file="${joint_limits_parameters_file}"
-      kinematics_parameters_file="${kinematics_parameters_file}"
-      physical_parameters_file="${physical_parameters_file}"
-      visual_parameters_file="${visual_parameters_file}"
-      force_abs_paths="${sim_gazebo or sim_ignition}"/> -->
+   <xacro:if value="$(arg sim_gazebo)">
+    <!-- Gazebo plugins -->
+    <gazebo reference="world">
+    </gazebo>
+    <gazebo>
+      <plugin filename="libgazebo_ros2_control.so" name="gazebo_ros2_control">
+        <parameters>$(arg simulation_controllers)</parameters>
+      </plugin>
+    </gazebo>
+  </xacro:if>
+  <xacro:if value="$(arg sim_ignition)">
+    <!-- Gazebo plugins -->
+    <gazebo reference="world">
+    </gazebo>
+    <gazebo>
+      <plugin filename="libign_ros2_control-system.so" name="ign_ros2_control::IgnitionROS2ControlPlugin">
+        <parameters>$(arg simulation_controllers)</parameters>
+        <controller_manager_node_name>$(arg prefix)controller_manager</controller_manager_node_name>
+      </plugin>
+    </gazebo>
+  </xacro:if>
 </robot>
