Commit message: fix: debug

File: src/ur3e_hande_robot_description/urdf/hande_extension.urdf.xacro (robot description, xacro)
@@ -113,116 +113,2 @@
   </xacro:if>
 </robot>
-<?xml version="1.0"?>
-<robot xmlns:xacro="http://wiki.ros.org/xacro" name="$(arg name)">
-   <!-- robot name parameter -->
-   <xacro:arg name="name" default="ur"/>
-   <!-- import main macro -->
-   <xacro:include filename="$(find ur_description)/urdf/ur_macro.xacro"/>
-   <!-- possible 'ur_type' values: ur3, ur3e, ur5, ur5e, ur10, ur10e, ur16e, ur20 -->
-   <!-- the default value should raise an error in case this was called without defining the type -->
-   <xacro:arg name="ur_type" default="ur5x"/>
-   <!-- parameters -->
-   <xacro:arg name="tf_prefix" default="" />
-   <xacro:arg name="joint_limit_params" default="$(find ur_description)/config/$(arg ur_type)/joint_limits.yaml"/>
-   <xacro:arg name="kinematics_params" default="$(find ur_description)/config/$(arg ur_type)/default_kinematics.yaml"/>
-   <xacro:arg name="physical_params" default="$(find ur_description)/config/$(arg ur_type)/physical_parameters.yaml"/>
-   <xacro:arg name="visual_params" default="$(find ur_description)/config/$(arg ur_type)/visual_parameters.yaml"/>
-   <xacro:arg name="transmission_hw_interface" default=""/>
-   <xacro:arg name="safety_limits" default="false"/>
-   <xacro:arg name="safety_pos_margin" default="0.15"/>
-   <xacro:arg name="safety_k_position" default="20"/>
-   <!-- ros2_control related parameters -->
-   <xacro:arg name="headless_mode" default="false" />
-   <xacro:arg name="robot_ip" default="0.0.0.0" />
-   <xacro:arg name="script_filename" default=""/>
-   <xacro:arg name="output_recipe_filename" default=""/>
-   <xacro:arg name="input_recipe_filename" default=""/>
-   <xacro:arg name="reverse_ip" default="0.0.0.0"/>
-   <xacro:arg name="script_command_port" default="50004"/>
-   <xacro:arg name="reverse_port" default="50001"/>
-   <xacro:arg name="script_sender_port" default="50002"/>
-   <xacro:arg name="trajectory_port" default="50003"/>
-   <!--   tool communication related parameters-->
-   <xacro:arg name="use_tool_communication" default="false" />
-   <xacro:arg name="tool_voltage" default="0" />
-   <xacro:arg name="tool_parity" default="0" />
-   <xacro:arg name="tool_baud_rate" default="115200" />
-   <xacro:arg name="tool_stop_bits" default="1" />
-   <xacro:arg name="tool_rx_idle_chars" default="1.5" />
-   <xacro:arg name="tool_tx_idle_chars" default="3.5" />
-   <xacro:arg name="tool_device_name" default="/tmp/ttyUR" />
-   <xacro:arg name="tool_tcp_port" default="54321" />
-     <!-- Simulation parameters -->
-   <xacro:arg name="use_fake_hardware" default="false" />
-   <xacro:arg name="fake_sensor_commands" default="false" />
-   <xacro:arg name="sim_gazebo" default="false" />
-   <xacro:arg name="sim_ignition" default="false" />
-   <xacro:arg name="simulation_controllers" default="" />
-   <!-- initial position for simulations (Fake Hardware, Gazebo, Ignition) -->
-   <xacro:arg name="initial_positions_file" default="$(find ur_description)/config/initial_positions.yaml"/>
-   <!-- convert to property to use substitution in function -->
-   <xacro:property name="initial_positions_file" default="$(arg initial_positions_file)"/>
-   <!-- create link fixed to the "world" -->
-   <link name="world" />
-   <!-- arm -->
-   <xacro:ur_robot
-     name="$(arg name)"
-     tf_prefix="$(arg tf_prefix)"
-     parent="world"
-     joint_limits_parameters_file="$(arg joint_limit_params)"
-     kinematics_parameters_file="$(arg kinematics_params)"
-     physical_parameters_file="$(arg physical_params)"
-     visual_parameters_file="$(arg visual_params)"
-     transmission_hw_interface="$(arg transmission_hw_interface)"
-     safety_limits="$(arg safety_limits)"
-     safety_pos_margin="$(arg safety_pos_margin)"
-     safety_k_position="$(arg safety_k_position)"
-     use_fake_hardware="$(arg use_fake_hardware)"
-     fake_sensor_commands="$(arg fake_sensor_commands)"
-     sim_gazebo="$(arg sim_gazebo)"
-     sim_ignition="$(arg sim_ignition)"
-     headless_mode="$(arg headless_mode)"
-     initial_positions="${xacro.load_yaml(initial_positions_file)}"
-     use_tool_communication="$(arg use_tool_communication)"
-     tool_voltage="$(arg tool_voltage)"
-     tool_parity="$(arg tool_parity)"
-     tool_baud_rate="$(arg tool_baud_rate)"
-     tool_stop_bits="$(arg tool_stop_bits)"
-     tool_rx_idle_chars="$(arg tool_rx_idle_chars)"
-     tool_tx_idle_chars="$(arg tool_tx_idle_chars)"
-     tool_device_name="$(arg tool_device_name)"
-     tool_tcp_port="$(arg tool_tcp_port)"
-     robot_ip="$(arg robot_ip)"
-     script_filename="$(arg script_filename)"
-     output_recipe_filename="$(arg output_recipe_filename)"
-     input_recipe_filename="$(arg input_recipe_filename)"
-     reverse_ip="$(arg reverse_ip)"
-     script_command_port="$(arg script_command_port)"
-     reverse_port="$(arg reverse_port)"
-     script_sender_port="$(arg script_sender_port)"
-     trajectory_port="$(arg trajectory_port)"
-     >
-     <origin xyz="0 0 0" rpy="0 0 0" />          <!-- position robot in the world -->
-   </xacro:ur_robot>
-   <xacro:if value="$(arg sim_gazebo)">
-    <!-- Gazebo plugins -->
-    <gazebo reference="world">
-    </gazebo>
-    <gazebo>
-      <plugin filename="libgazebo_ros2_control.so" name="gazebo_ros2_control">
-        <parameters>$(arg simulation_controllers)</parameters>
-      </plugin>
-    </gazebo>
-  </xacro:if>
-  <xacro:if value="$(arg sim_ignition)">
-    <!-- Gazebo plugins -->
-    <gazebo reference="world">
-    </gazebo>
-    <gazebo>
-      <plugin filename="libign_ros2_control-system.so" name="ign_ros2_control::IgnitionROS2ControlPlugin">
-        <parameters>$(arg simulation_controllers)</parameters>
-        <controller_manager_node_name>$(arg tf_prefix)controller_manager</controller_manager_node_name>
-      </plugin>
-    </gazebo>
-  </xacro:if>
-</robot>

Commit message: fix: add link

File: src/ur3e_hande_robot_description/urdf/hande_extension.urdf.xacro (robot description, xacro)
@@ -90,6 +90,4 @@
      trajectory_port="$(arg trajectory_port)"
      >
-     <origin xyz="0 0 0" rpy="0 0 0" />          <!-- position robot in the world -->
-   </xacro:ur_robot>
     <xacro:robotiq_hande
      name="$(arg name)"
@@ -97,4 +95,11 @@
      ur_type="$(arg ur_type)"
    />
+    <joint name="${tf_prefix}hande_to_wrist_flange" type="fixed">
+      <parent link="${tf_prefix}flange" />
+      <child link="${tf_prefix}robotiq_hande_base_link" />
+      <origin xyz="0 0 0" rpy="0 0 0" />
+    </joint>
+     <origin xyz="0 0 0" rpy="0 0 0" />          <!-- position robot in the world -->
+   </xacro:ur_robot>
    <xacro:if value="$(arg sim_gazebo)">
     <!-- Gazebo plugins -->

Commit message: fix: debug

File: src/ur3e_hande_robot_description/urdf/hande_extension.urdf.xacro (robot description, xacro)
@@ -95,7 +95,7 @@
      ur_type="$(arg ur_type)"
    />
-    <joint name="${tf_prefix}hande_to_wrist_flange" type="fixed">
-      <parent link="${tf_prefix}flange" />
-      <child link="${tf_prefix}robotiq_hande_base_link" />
+    <joint name="$(arg tf_prefix)hande_to_wrist_flange" type="fixed">
+      <parent link="$(arg tf_prefix)flange" />
+      <child link="$(arg tf_prefix)robotiq_hande_base_link" />
       <origin xyz="0 0 0" rpy="0 0 0" />
     </joint>

Commit message: fix: debug

File: src/ur3e_hande_robot_description/urdf/hande_extension.urdf.xacro (robot description, xacro)
@@ -96,5 +96,5 @@
    />
     <joint name="$(arg tf_prefix)hande_to_wrist_flange" type="fixed">
-      <parent link="$(arg tf_prefix)flange" />
+      <parent link="$(arg tf_prefix)tool0" />
       <child link="$(arg tf_prefix)robotiq_hande_base_link" />
       <origin xyz="0 0 0" rpy="0 0 0" />

Commit message: fix: bugs

File: src/ur3e_hande_robot_description/urdf/hande_extension.urdf.xacro (robot description, xacro)
@@ -99,5 +99,5 @@
    />
     <joint name="$(arg tf_prefix)hande_to_wrist_flange" type="fixed">
-      <parent link="world" />
+      <parent link="$(arg tf_prefix)flange" />
       <child link="$(arg tf_prefix)robotiq_hande_base_link" />
       <origin xyz="1 1 0" rpy="0 0 0" />

Commit message: fix: correct hande joint orientation

File: src/ur3e_hande_robot_description/urdf/hande_extension.urdf.xacro (robot description, xacro)
@@ -101,5 +101,5 @@
       <parent link="$(arg tf_prefix)flange" />
       <child link="$(arg tf_prefix)robotiq_hande_base_link" />
-      <origin xyz="1 1 0" rpy="0 0 0" />
+      <origin xyz="0 0 0" rpy="${pi/2.0} 0 ${pi/2.0}" />
     </joint>
    <xacro:if value="$(arg sim_gazebo)">
