Commit message: fix: correct grasping point

File: src/ur3e_hande_robot_description/urdf/hande_black.xacro (robot description, xacro)
@@ -141,5 +141,5 @@
     </joint>
     <joint name="${tf_prefix}grasping_point" type="fixed">
-      <origin rpy="0 0 0" xyz="0.0 0.0 0.15"/>
+      <origin rpy="0 0 0" xyz="0.0 0.0 0.095"/>
       <parent link="${tf_prefix}robotiq_hande_base_link"/>
       <child link="grasping_point_link"/>

Commit message: fix: correct urdfs + aruco

File: src/ur3e_hande_robot_description/urdf/hande_black.xacro (robot description, xacro)
@@ -38,5 +38,5 @@
     <link name="${tf_prefix}robotiq_coupler">
       <inertial>
-        <mass value="0.168" />
+        <mass value="0.100" />
         <inertia
           ixx="6.17674E-05" ixy="0.0" ixz="0.0"
@@ -74,7 +74,13 @@
         </geometry>
       </collision>
-      <xacro:cylinder_inertial radius="${hande_base_inertia_radius}" length="${hande_base_inertia_length}"  mass="${hande_base_mass}">
+      <inertia
+          ixx="0.005341" ixy="0.0" ixz="0.0"
+          iyx="0.0"  iyy="0.005447" iyz="0.0"
+          izx="0.0"  izy="0.0" izz="0.000636"
+        />
+      </inertial>
+      <!-- <xacro:cylinder_inertial radius="${hande_base_inertia_radius}" length="${hande_base_inertia_length}"  mass="${hande_base_mass}">
         <origin xyz="0.0 0.0 ${-0.5 * hande_base_inertia_length}" rpy="0 0 0" />
-      </xacro:cylinder_inertial>
+      </xacro:cylinder_inertial> -->
     </link>
     <link name="${tf_prefix}left_finger">
@@ -94,7 +100,7 @@
         </geometry>
       </collision>
-      <xacro:cylinder_inertial radius="${left_finger_inertia_radius}" length="${left_finger_inertia_length}"  mass="${left_finger_mass}">
+      <!-- <xacro:cylinder_inertial radius="${left_finger_inertia_radius}" length="${left_finger_inertia_length}"  mass="${left_finger_mass}">
         <origin xyz="0.0 0.0 ${-0.5 * left_finger_inertia_length}" rpy="0 0 0" />
-      </xacro:cylinder_inertial>
+      </xacro:cylinder_inertial> -->
     </link>
     <link name="${tf_prefix}right_finger">
@@ -114,7 +120,7 @@
         </geometry>
       </collision>
-      <xacro:cylinder_inertial radius="${right_finger_inertia_radius}" length="${right_finger_inertia_length}"  mass="${right_finger_mass}">
+      <!-- <xacro:cylinder_inertial radius="${right_finger_inertia_radius}" length="${right_finger_inertia_length}"  mass="${right_finger_mass}">
         <origin xyz="0.0 0.0 ${-0.5 * right_finger_inertia_length}" rpy="0 0 0" />
-      </xacro:cylinder_inertial>
+      </xacro:cylinder_inertial> -->
     </link>
     <link name="grasping_point_link">

Commit message: fix: correct urdf

File: src/ur3e_hande_robot_description/urdf/hande_black.xacro (robot description, xacro)
@@ -74,13 +74,14 @@
         </geometry>
       </collision>
-      <inertia
-          ixx="0.005341" ixy="0.0" ixz="0.0"
-          iyx="0.0"  iyy="0.005447" iyz="0.0"
-          izx="0.0"  izy="0.0" izz="0.000636"
+            <!-- <inertial>
+        <inertial
+            ixx="0.005341" ixy="0.0" ixz="0.0"
+            iyy="0.005447" iyz="0.0"
+            izz="0.000636"
         />
-      </inertial>
-      <!-- <xacro:cylinder_inertial radius="${hande_base_inertia_radius}" length="${hande_base_inertia_length}"  mass="${hande_base_mass}">
+      </inertial> -->
+      <xacro:cylinder_inertial radius="${hande_base_inertia_radius}" length="${hande_base_inertia_length}"  mass="${hande_base_mass}">
         <origin xyz="0.0 0.0 ${-0.5 * hande_base_inertia_length}" rpy="0 0 0" />
-      </xacro:cylinder_inertial> -->
+      </xacro:cylinder_inertial>
     </link>
     <link name="${tf_prefix}left_finger">
@@ -100,7 +101,7 @@
         </geometry>
       </collision>
-      <!-- <xacro:cylinder_inertial radius="${left_finger_inertia_radius}" length="${left_finger_inertia_length}"  mass="${left_finger_mass}">
+      <xacro:cylinder_inertial radius="${left_finger_inertia_radius}" length="${left_finger_inertia_length}"  mass="${left_finger_mass}">
         <origin xyz="0.0 0.0 ${-0.5 * left_finger_inertia_length}" rpy="0 0 0" />
-      </xacro:cylinder_inertial> -->
+      </xacro:cylinder_inertial>
     </link>
     <link name="${tf_prefix}right_finger">
@@ -120,7 +121,7 @@
         </geometry>
       </collision>
-      <!-- <xacro:cylinder_inertial radius="${right_finger_inertia_radius}" length="${right_finger_inertia_length}"  mass="${right_finger_mass}">
+      <xacro:cylinder_inertial radius="${right_finger_inertia_radius}" length="${right_finger_inertia_length}"  mass="${right_finger_mass}">
         <origin xyz="0.0 0.0 ${-0.5 * right_finger_inertia_length}" rpy="0 0 0" />
-      </xacro:cylinder_inertial> -->
+      </xacro:cylinder_inertial>
     </link>
     <link name="grasping_point_link">

Commit message: fix: adjust grasping point

File: src/ur3e_hande_robot_description/urdf/hande_black.xacro (robot description, xacro)
@@ -141,5 +141,5 @@
     </joint>
     <joint name="${tf_prefix}grasping_point" type="fixed">
-      <origin rpy="0 0 0" xyz="0.0 0.0 0.095"/>
+      <origin rpy="0 0 0" xyz="0.0 0.0 0.09"/>
       <parent link="${tf_prefix}robotiq_hande_base_link"/>
       <child link="grasping_point_link"/>
