Commit message: fix: xacro init pos

File: src/ur3e_hande_robot_description/urdf/hande.xacro (robot description, xacro)
@@ -47,6 +47,5 @@
     kinematics_parameters_file
     physical_parameters_file
-    visual_parameters_file
-    initial_positions:=${dict(joint_finger=0.01,robotiq_hande_base_to_right_finger=0.01)}" >
+    visual_parameters_file" >
     <!-- customization to include hande -->
     <link name="${prefix}robotiq_hande_base_link">

File: src/ur3e_hande_robot_description/urdf/hande_extension.urdf.xacro (robot description, xacro)
@@ -50,5 +50,4 @@
      physical_parameters_file="$(arg hande_physical_params)"
      visual_parameters_file="$(arg hande_visual_params)"
-     initial_positions="${xacro.load_yaml(initial_positions_file)}"
    />
     <!-- name
@@ -62,4 +61,6 @@
     initial_positions:=${dict(joint_finger=0.01,robotiq_hande_base_to_right_finger=0.01)}" >
   -->
+   <!-- create link fixed to the "world" -->
+   <link name="world" />
    <xacro:ur_robot
      name="$(arg name)"
@@ -96,9 +97,10 @@
      script_command_port="$(arg script_command_port)"
      >
+<!--
     <joint name="${prefix}hande_to_wrist_flange" type="fixed">
       <parent link="${prefix}flange" />
       <child link="${prefix}robotiq_hande_base_link" />
       <origin xyz="0 0 0" rpy="0 0 0" />
-    </joint>
+    </joint> -->
      <origin xyz="0 0 0" rpy="0 0 0" />          <!-- position robot in the world -->
    </xacro:ur_robot>

Commit message: fix: debug steps

File: src/ur3e_hande_robot_description/urdf/hande.xacro (robot description, xacro)
@@ -2,8 +2,8 @@
 <robot xmlns:xacro="http://wiki.ros.org/xacro" name="$(arg name)">
   <xacro:arg name="name" default="hande"/>
-  <xacro:property name="hande_joint_limit_params" value="$(find ur3e_hande_robot_description)/config/hande/joint_limits.yaml"/>
-  <xacro:property name="hande_kinematics_params" value="$(find ur3e_hande_robot_description)/config/hande/default_kinematics.yaml"/>
-  <xacro:property name="hande_physical_params" value="$(find ur3e_hande_robot_description)/config/hande/physical_parameters.yaml"/>
-  <xacro:property name="hande_visual_params" value="$(find ur3e_hande_robot_description)/config/hande/visual_parameters.yaml"/>
+  <xacro:property name="hande_joint_limit_params" value="$(find ur3e_hande_robot_description)/config/$(arg ur_type)/joint_limits.yaml"/>
+  <xacro:property name="hande_kinematics_params" value="$(find ur3e_hande_robot_description)/config/$(arg ur_type)/default_kinematics.yaml"/>
+  <xacro:property name="hande_physical_params" value="$(find ur3e_hande_robot_description)/config/$(arg ur_type)/physical_parameters.yaml"/>
+  <xacro:property name="hande_visual_params" value="$(find ur3e_hande_robot_description)/config/$(arg ur_type)/visual_parameters.yaml"/>
   <xacro:macro name="cylinder_inertial" params="radius length mass *origin">
     <inertial>

File: src/ur3e_hande_robot_description/urdf/hande_extension.urdf.xacro (robot description, xacro)
@@ -2,5 +2,5 @@
 <robot xmlns:xacro="http://wiki.ros.org/xacro" name="$(arg name)">
   <xacro:include filename="$(find ur_description)/urdf/ur_macro.xacro"/>
-  <xacro:include filename="$(find ur3e_hande_robot_description)/urdf/hande.xacro"/>
+  <!-- <xacro:include filename="$(find ur3e_hande_robot_description)/urdf/hande.xacro"/> -->
    <xacro:arg name="ur_type" default="ur5x"/>
    <!-- parameters -->
@@ -42,5 +42,5 @@
    <xacro:arg name="sim_ignition" default="false" />
    <xacro:arg name="simulation_controllers" default="" />
-    <xacro:robotiq_hande
+    <!-- <xacro:robotiq_hande
      name="$(arg name)"
      prefix="$(arg prefix)"
@@ -50,5 +50,5 @@
      physical_parameters_file="$(arg hande_physical_params)"
      visual_parameters_file="$(arg hande_visual_params)"
-   />
+   /> -->
     <!-- name
     prefix

Commit message: fix: debugging

File: src/ur3e_hande_robot_description/urdf/hande.xacro (robot description, xacro)
@@ -39,4 +39,5 @@
   <xacro:property name="hande_base_radius" value="${sec_inertia_parameters['hande_base_radius']}" scope="parent"/>
   <xacro:property name="finger_radius" value="${sec_inertia_parameters['finger_radius']}" scope="parent"/>
+<!--
 <xacro:macro name="robotiq_hande" params="
     name
@@ -147,4 +148,4 @@
       <origin xyz="0 0 0" rpy="0 ${-pi/2.0} ${-pi/2.0}" />
     </joint> -->
-</xacro:macro>
+</xacro:macro> -->
 </robot>

File: src/ur3e_hande_robot_description/urdf/hande_extension.urdf.xacro (robot description, xacro)
@@ -4,14 +4,14 @@
    <xacro:arg name="name" default="ur"/>
    <!-- import main macro -->
-   <xacro:include filename="$(find ur3e_hande_robot_description)/urdf/ur_macro.xacro"/>
-   <!-- possible 'ur_type' values: ur3, ur3e, ur5, ur5e, ur10, ur10e, ur16e -->
+   <xacro:include filename="$(find ur_description)/urdf/ur_macro.xacro"/>
+   <!-- possible 'ur_type' values: ur3, ur3e, ur5, ur5e, ur10, ur10e, ur16e, ur20 -->
    <!-- the default value should raise an error in case this was called without defining the type -->
    <xacro:arg name="ur_type" default="ur5x"/>
    <!-- parameters -->
-   <xacro:arg name="prefix" default="" />
-   <xacro:arg name="joint_limit_params" default="$(find ur3e_hande_robot_description)/config/$(arg ur_type)/joint_limits.yaml"/>
-   <xacro:arg name="kinematics_params" default="$(find ur3e_hande_robot_description)/config/$(arg ur_type)/default_kinematics.yaml"/>
-   <xacro:arg name="physical_params" default="$(find ur3e_hande_robot_description)/config/$(arg ur_type)/physical_parameters.yaml"/>
-   <xacro:arg name="visual_params" default="$(find ur3e_hande_robot_description)/config/$(arg ur_type)/visual_parameters.yaml"/>
+   <xacro:arg name="tf_prefix" default="" />
+   <xacro:arg name="joint_limit_params" default="$(find ur_description)/config/$(arg ur_type)/joint_limits.yaml"/>
+   <xacro:arg name="kinematics_params" default="$(find ur_description)/config/$(arg ur_type)/default_kinematics.yaml"/>
+   <xacro:arg name="physical_params" default="$(find ur_description)/config/$(arg ur_type)/physical_parameters.yaml"/>
+   <xacro:arg name="visual_params" default="$(find ur_description)/config/$(arg ur_type)/visual_parameters.yaml"/>
    <xacro:arg name="transmission_hw_interface" default=""/>
    <xacro:arg name="safety_limits" default="false"/>
@@ -26,4 +26,7 @@
    <xacro:arg name="reverse_ip" default="0.0.0.0"/>
    <xacro:arg name="script_command_port" default="50004"/>
+   <xacro:arg name="reverse_port" default="50001"/>
+   <xacro:arg name="script_sender_port" default="50002"/>
+   <xacro:arg name="trajectory_port" default="50003"/>
    <!--   tool communication related parameters-->
    <xacro:arg name="use_tool_communication" default="false" />
@@ -43,5 +46,5 @@
    <xacro:arg name="simulation_controllers" default="" />
    <!-- initial position for simulations (Fake Hardware, Gazebo, Ignition) -->
-   <xacro:arg name="initial_positions_file" default="$(find ur3e_hande_robot_description)/config/initial_positions.yaml"/>
+   <xacro:arg name="initial_positions_file" default="$(find ur_description)/config/initial_positions.yaml"/>
    <!-- convert to property to use substitution in function -->
    <xacro:property name="initial_positions_file" default="$(arg initial_positions_file)"/>
@@ -51,5 +54,5 @@
    <xacro:ur_robot
      name="$(arg name)"
-     prefix="$(arg prefix)"
+     tf_prefix="$(arg tf_prefix)"
      parent="world"
      joint_limits_parameters_file="$(arg joint_limit_params)"
@@ -82,4 +85,7 @@
      reverse_ip="$(arg reverse_ip)"
      script_command_port="$(arg script_command_port)"
+     reverse_port="$(arg reverse_port)"
+     script_sender_port="$(arg script_sender_port)"
+     trajectory_port="$(arg trajectory_port)"
      >
      <origin xyz="0 0 0" rpy="0 0 0" />          <!-- position robot in the world -->
@@ -102,7 +108,121 @@
       <plugin filename="libign_ros2_control-system.so" name="ign_ros2_control::IgnitionROS2ControlPlugin">
         <parameters>$(arg simulation_controllers)</parameters>
-        <controller_manager_node_name>$(arg prefix)controller_manager</controller_manager_node_name>
+        <controller_manager_node_name>$(arg tf_prefix)controller_manager</controller_manager_node_name>
       </plugin>
     </gazebo>
   </xacro:if>
 </robot>
+<?xml version="1.0"?>
+<robot xmlns:xacro="http://wiki.ros.org/xacro" name="$(arg name)">
+   <!-- robot name parameter -->
+   <xacro:arg name="name" default="ur"/>
+   <!-- import main macro -->
+   <xacro:include filename="$(find ur_description)/urdf/ur_macro.xacro"/>
+   <!-- possible 'ur_type' values: ur3, ur3e, ur5, ur5e, ur10, ur10e, ur16e, ur20 -->
+   <!-- the default value should raise an error in case this was called without defining the type -->
+   <xacro:arg name="ur_type" default="ur5x"/>
+   <!-- parameters -->
+   <xacro:arg name="tf_prefix" default="" />
+   <xacro:arg name="joint_limit_params" default="$(find ur_description)/config/$(arg ur_type)/joint_limits.yaml"/>
+   <xacro:arg name="kinematics_params" default="$(find ur_description)/config/$(arg ur_type)/default_kinematics.yaml"/>
+   <xacro:arg name="physical_params" default="$(find ur_description)/config/$(arg ur_type)/physical_parameters.yaml"/>
+   <xacro:arg name="visual_params" default="$(find ur_description)/config/$(arg ur_type)/visual_parameters.yaml"/>
+   <xacro:arg name="transmission_hw_interface" default=""/>
+   <xacro:arg name="safety_limits" default="false"/>
+   <xacro:arg name="safety_pos_margin" default="0.15"/>
+   <xacro:arg name="safety_k_position" default="20"/>
+   <!-- ros2_control related parameters -->
+   <xacro:arg name="headless_mode" default="false" />
+   <xacro:arg name="robot_ip" default="0.0.0.0" />
+   <xacro:arg name="script_filename" default=""/>
+   <xacro:arg name="output_recipe_filename" default=""/>
+   <xacro:arg name="input_recipe_filename" default=""/>
+   <xacro:arg name="reverse_ip" default="0.0.0.0"/>
+   <xacro:arg name="script_command_port" default="50004"/>
+   <xacro:arg name="reverse_port" default="50001"/>
+   <xacro:arg name="script_sender_port" default="50002"/>
+   <xacro:arg name="trajectory_port" default="50003"/>
+   <!--   tool communication related parameters-->
+   <xacro:arg name="use_tool_communication" default="false" />
+   <xacro:arg name="tool_voltage" default="0" />
+   <xacro:arg name="tool_parity" default="0" />
+   <xacro:arg name="tool_baud_rate" default="115200" />
+   <xacro:arg name="tool_stop_bits" default="1" />
+   <xacro:arg name="tool_rx_idle_chars" default="1.5" />
+   <xacro:arg name="tool_tx_idle_chars" default="3.5" />
+   <xacro:arg name="tool_device_name" default="/tmp/ttyUR" />
+   <xacro:arg name="tool_tcp_port" default="54321" />
+     <!-- Simulation parameters -->
+   <xacro:arg name="use_fake_hardware" default="false" />
+   <xacro:arg name="fake_sensor_commands" default="false" />
+   <xacro:arg name="sim_gazebo" default="false" />
+   <xacro:arg name="sim_ignition" default="false" />
+   <xacro:arg name="simulation_controllers" default="" />
+   <!-- initial position for simulations (Fake Hardware, Gazebo, Ignition) -->
+   <xacro:arg name="initial_positions_file" default="$(find ur_description)/config/initial_positions.yaml"/>
+   <!-- convert to property to use substitution in function -->
+   <xacro:property name="initial_positions_file" default="$(arg initial_positions_file)"/>
+   <!-- create link fixed to the "world" -->
+   <link name="world" />
+   <!-- arm -->
+   <xacro:ur_robot
+     name="$(arg name)"
+     tf_prefix="$(arg tf_prefix)"
+     parent="world"
+     joint_limits_parameters_file="$(arg joint_limit_params)"
+     kinematics_parameters_file="$(arg kinematics_params)"
+     physical_parameters_file="$(arg physical_params)"
+     visual_parameters_file="$(arg visual_params)"
+     transmission_hw_interface="$(arg transmission_hw_interface)"
+     safety_limits="$(arg safety_limits)"
+     safety_pos_margin="$(arg safety_pos_margin)"
+     safety_k_position="$(arg safety_k_position)"
+     use_fake_hardware="$(arg use_fake_hardware)"
+     fake_sensor_commands="$(arg fake_sensor_commands)"
+     sim_gazebo="$(arg sim_gazebo)"
+     sim_ignition="$(arg sim_ignition)"
+     headless_mode="$(arg headless_mode)"
+     initial_positions="${xacro.load_yaml(initial_positions_file)}"
+     use_tool_communication="$(arg use_tool_communication)"
+     tool_voltage="$(arg tool_voltage)"
+     tool_parity="$(arg tool_parity)"
+     tool_baud_rate="$(arg tool_baud_rate)"
+     tool_stop_bits="$(arg tool_stop_bits)"
+     tool_rx_idle_chars="$(arg tool_rx_idle_chars)"
+     tool_tx_idle_chars="$(arg tool_tx_idle_chars)"
+     tool_device_name="$(arg tool_device_name)"
+     tool_tcp_port="$(arg tool_tcp_port)"
+     robot_ip="$(arg robot_ip)"
+     script_filename="$(arg script_filename)"
+     output_recipe_filename="$(arg output_recipe_filename)"
+     input_recipe_filename="$(arg input_recipe_filename)"
+     reverse_ip="$(arg reverse_ip)"
+     script_command_port="$(arg script_command_port)"
+     reverse_port="$(arg reverse_port)"
+     script_sender_port="$(arg script_sender_port)"
+     trajectory_port="$(arg trajectory_port)"
+     >
+     <origin xyz="0 0 0" rpy="0 0 0" />          <!-- position robot in the world -->
+   </xacro:ur_robot>
+   <xacro:if value="$(arg sim_gazebo)">
+    <!-- Gazebo plugins -->
+    <gazebo reference="world">
+    </gazebo>
+    <gazebo>
+      <plugin filename="libgazebo_ros2_control.so" name="gazebo_ros2_control">
+        <parameters>$(arg simulation_controllers)</parameters>
+      </plugin>
+    </gazebo>
+  </xacro:if>
+  <xacro:if value="$(arg sim_ignition)">
+    <!-- Gazebo plugins -->
+    <gazebo reference="world">
+    </gazebo>
+    <gazebo>
+      <plugin filename="libign_ros2_control-system.so" name="ign_ros2_control::IgnitionROS2ControlPlugin">
+        <parameters>$(arg simulation_controllers)</parameters>
+        <controller_manager_node_name>$(arg tf_prefix)controller_manager</controller_manager_node_name>
+      </plugin>
+    </gazebo>
+  </xacro:if>
+</robot>

Commit message: fix: debug

File: src/ur3e_hande_robot_description/urdf/hande.xacro (robot description, xacro)
@@ -39,21 +39,9 @@
   <xacro:property name="hande_base_radius" value="${sec_inertia_parameters['hande_base_radius']}" scope="parent"/>
   <xacro:property name="finger_radius" value="${sec_inertia_parameters['finger_radius']}" scope="parent"/>
-<!--
 <xacro:macro name="robotiq_hande" params="
     name
-    prefix
-    parent
-    *origin
-    joint_limits_parameters_file
-    kinematics_parameters_file
-    physical_parameters_file
-    visual_parameters_file" >
+    prefix" >
     <!-- customization to include hande -->
     <link name="${prefix}robotiq_hande_base_link">
-<!--       <inertial>
-        <origin xyz="0 0 0.04607" rpy="0 0 0" />
-        <mass value="0.86387" />
-        <inertia ixx="1017560E-9" ixy="0" ixz="2235E-9" iyy="1028041E-9" iyz="0" izz="489810E-9" />
-      </inertial> -->
       <visual>
         <origin xyz="0 0 0" rpy="0 0 0" />
@@ -76,9 +64,4 @@
     </link>
     <link name="${prefix}left_finger">
-<!--       <inertial>
-        <origin rpy="0 0 0" xyz="0.02262 -0.00759 0.00738"/>
-        <mass value="0.03804"/>
-        <inertia ixx="13567E-9" ixy="1849E-9" ixz="3622E-9" iyy="15784E-9" iyz="3616E-9" izz="7478E-9"/>
-      </inertial> -->
       <visual>
         <origin rpy="0 0 0" xyz="0 0 0"/>
@@ -101,9 +84,4 @@
     </link>
     <link name="${prefix}right_finger">
-<!--       <inertial>
-        <origin rpy="0 0 0" xyz="-0.02262 0.00759 0.00738"/>
-        <mass value="0.03804"/>
-        <inertia ixx="13567E-9" ixy="1849E-9" ixz="-3622E-9" iyy="15784E-9" iyz="-3616E-9" izz="7478E-9"/>
-      </inertial> -->
       <visual>
         <origin rpy="0 0 0" xyz="0 0 0"/>
@@ -141,11 +119,4 @@
       <mimic joint="${prefix}joint_finger" multiplier="1" offset="0"/>
     </joint>
-    <!-- ROS-Industrial 'flange' frame - attachment point for EEF models -->
-    <!-- <link name="${prefix}flange" />
-    <joint name="${prefix}wrist_3-flange" type="fixed">
-      <parent link="${prefix}wrist_3_link" />
-      <child link="${prefix}flange" />
-      <origin xyz="0 0 0" rpy="0 ${-pi/2.0} ${-pi/2.0}" />
-    </joint> -->
-</xacro:macro> -->
+</xacro:macro>
 </robot>

File: src/ur3e_hande_robot_description/urdf/hande_extension.urdf.xacro (robot description, xacro)
@@ -92,4 +92,8 @@
      <origin xyz="0 0 0" rpy="0 0 0" />          <!-- position robot in the world -->
    </xacro:ur_robot>
+    <xacro:robotiq_hande
+     name="$(arg name)"
+     prefix="$(arg prefix)"
+   />
    <xacro:if value="$(arg sim_gazebo)">
     <!-- Gazebo plugins -->

Commit message: fix: debug

File: src/ur3e_hande_robot_description/urdf/hande.xacro (robot description, xacro)
@@ -2,4 +2,8 @@
 <robot xmlns:xacro="http://wiki.ros.org/xacro" name="$(arg name)">
   <xacro:arg name="name" default="hande"/>
+<xacro:macro name="robotiq_hande" params="
+    name
+    prefix
+    ur_type" >
   <xacro:property name="hande_joint_limit_params" value="$(find ur3e_hande_robot_description)/config/$(arg ur_type)/joint_limits.yaml"/>
   <xacro:property name="hande_kinematics_params" value="$(find ur3e_hande_robot_description)/config/$(arg ur_type)/default_kinematics.yaml"/>
@@ -39,7 +43,4 @@
   <xacro:property name="hande_base_radius" value="${sec_inertia_parameters['hande_base_radius']}" scope="parent"/>
   <xacro:property name="finger_radius" value="${sec_inertia_parameters['finger_radius']}" scope="parent"/>
-<xacro:macro name="robotiq_hande" params="
-    name
-    prefix" >
     <!-- customization to include hande -->
     <link name="${prefix}robotiq_hande_base_link">

File: src/ur3e_hande_robot_description/urdf/hande_extension.urdf.xacro (robot description, xacro)
@@ -95,4 +95,5 @@
      name="$(arg name)"
      prefix="$(arg prefix)"
+     ur_type="$(arg ur_type)"
    />
    <xacro:if value="$(arg sim_gazebo)">

Commit message: fix: debug

File: src/ur3e_hande_robot_description/urdf/hande.xacro (robot description, xacro)
@@ -4,5 +4,5 @@
 <xacro:macro name="robotiq_hande" params="
     name
-    prefix
+    tf_prefix
     ur_type" >
   <xacro:property name="hande_joint_limit_params" value="$(find ur3e_hande_robot_description)/config/$(arg ur_type)/joint_limits.yaml"/>
@@ -44,5 +44,5 @@
   <xacro:property name="finger_radius" value="${sec_inertia_parameters['finger_radius']}" scope="parent"/>
     <!-- customization to include hande -->
-    <link name="${prefix}robotiq_hande_base_link">
+    <link name="${tf_prefix}robotiq_hande_base_link">
       <visual>
         <origin xyz="0 0 0" rpy="0 0 0" />
@@ -64,5 +64,5 @@
       </xacro:cylinder_inertial>
     </link>
-    <link name="${prefix}left_finger">
+    <link name="${tf_prefix}left_finger">
       <visual>
         <origin rpy="0 0 0" xyz="0 0 0"/>
@@ -84,5 +84,5 @@
       </xacro:cylinder_inertial>
     </link>
-    <link name="${prefix}right_finger">
+    <link name="${tf_prefix}right_finger">
       <visual>
         <origin rpy="0 0 0" xyz="0 0 0"/>
@@ -105,18 +105,18 @@
     </link>
     <!-- hande installation -->
-    <joint name="${prefix}joint_finger" type="prismatic">
+    <joint name="${tf_prefix}joint_finger" type="prismatic">
       <origin rpy="0 0 0" xyz="0 0 0.099"/>
-      <parent link="${prefix}robotiq_hande_base_link"/>
-      <child link="${prefix}left_finger"/>
+      <parent link="${tf_prefix}robotiq_hande_base_link"/>
+      <child link="${tf_prefix}left_finger"/>
       <axis xyz="-1 0 0"/>
       <limit effort="130" lower="0" upper="0.025" velocity="0.15"/>
     </joint>
-    <joint name="robotiq_hande_base_to_${prefix}right_finger" type="prismatic">
+    <joint name="robotiq_hande_base_to_${tf_prefix}right_finger" type="prismatic">
       <origin rpy="0 0 0" xyz="0 0 0.099"/>
-      <parent link="${prefix}robotiq_hande_base_link"/>
-      <child link="${prefix}right_finger"/>
+      <parent link="${tf_prefix}robotiq_hande_base_link"/>
+      <child link="${tf_prefix}right_finger"/>
       <axis xyz="1 0 0"/>
       <limit effort="130" lower="0" upper="0.025" velocity="0.15"/>
-      <mimic joint="${prefix}joint_finger" multiplier="1" offset="0"/>
+      <mimic joint="${tf_prefix}joint_finger" multiplier="1" offset="0"/>
     </joint>
 </xacro:macro>

File: src/ur3e_hande_robot_description/urdf/hande_extension.urdf.xacro (robot description, xacro)
@@ -94,5 +94,5 @@
     <xacro:robotiq_hande
      name="$(arg name)"
-     prefix="$(arg prefix)"
+     tf_prefix="$(arg tf_prefix)"
      ur_type="$(arg ur_type)"
    />

Commit message: fix: bugs

File: src/ur3e_hande_robot_description/urdf/hande.xacro (robot description, xacro)
@@ -120,4 +120,9 @@
       <mimic joint="${tf_prefix}joint_finger" multiplier="1" offset="0"/>
     </joint>
+    <joint name="$(arg tf_prefix)hande_to_wrist_flange" type="fixed">
+      <parent link="world" />
+      <child link="$(arg tf_prefix)robotiq_hande_base_link" />
+      <origin xyz="0 0 0" rpy="0 0 0" />
+    </joint>
 </xacro:macro>
 </robot>

File: src/ur3e_hande_robot_description/urdf/hande_extension.urdf.xacro (robot description, xacro)
@@ -95,9 +95,4 @@
      ur_type="$(arg ur_type)"
    />
-    <joint name="$(arg tf_prefix)hande_to_wrist_flange" type="fixed">
-      <parent link="$(arg tf_prefix)tool0" />
-      <child link="$(arg tf_prefix)robotiq_hande_base_link" />
-      <origin xyz="0 0 0" rpy="0 0 0" />
-    </joint>
      <origin xyz="0 0 0" rpy="0 0 0" />          <!-- position robot in the world -->
    </xacro:ur_robot>

Commit message: fix: bug

File: src/ur3e_hande_robot_description/urdf/hande.xacro (robot description, xacro)
@@ -5,5 +5,6 @@
     name
     tf_prefix
-    ur_type" >
+    ur_type
+    parent" >
   <xacro:property name="hande_joint_limit_params" value="$(find ur3e_hande_robot_description)/config/$(arg ur_type)/joint_limits.yaml"/>
   <xacro:property name="hande_kinematics_params" value="$(find ur3e_hande_robot_description)/config/$(arg ur_type)/default_kinematics.yaml"/>
@@ -121,7 +122,7 @@
     </joint>
     <joint name="$(arg tf_prefix)hande_to_wrist_flange" type="fixed">
-      <parent link="world" />
-      <child link="$(arg tf_prefix)robotiq_hande_base_link" />
-      <origin xyz="0 0 0" rpy="0 0 0" />
+      <parent link="${parent}" />
+      <child link="${tf_prefix}robotiq_hande_base_link" />
+      <origin xyz="1 1 0" rpy="0 0 0" />
     </joint>
 </xacro:macro>

File: src/ur3e_hande_robot_description/urdf/hande_extension.urdf.xacro (robot description, xacro)
@@ -90,11 +90,12 @@
      trajectory_port="$(arg trajectory_port)"
      >
+     <origin xyz="0 0 0" rpy="0 0 0" />          <!-- position robot in the world -->
+   </xacro:ur_robot>
     <xacro:robotiq_hande
      name="$(arg name)"
      tf_prefix="$(arg tf_prefix)"
      ur_type="$(arg ur_type)"
+     parent="world"
    />
-     <origin xyz="0 0 0" rpy="0 0 0" />          <!-- position robot in the world -->
-   </xacro:ur_robot>
    <xacro:if value="$(arg sim_gazebo)">
     <!-- Gazebo plugins -->
