Commit message: fix: bugs bugs bugs

File: src/ur3e_hande_robot_description/urdf/hande.xacro (robot description, xacro)
@@ -121,9 +121,9 @@
       <mimic joint="${tf_prefix}joint_finger" multiplier="1" offset="0"/>
     </joint>
-    <joint name="$(arg tf_prefix)hande_to_wrist_flange" type="fixed">
+    <!-- <joint name="$(arg tf_prefix)hande_to_wrist_flange" type="fixed">
       <parent link="${parent}" />
       <child link="${tf_prefix}robotiq_hande_base_link" />
       <origin xyz="1 1 0" rpy="0 0 0" />
-    </joint>
+    </joint> -->
 </xacro:macro>
 </robot>

File: src/ur3e_hande_robot_description/urdf/hande_extension.urdf.xacro (robot description, xacro)
@@ -98,4 +98,9 @@
      parent="world"
    />
+    <joint name="$(arg tf_prefix)hande_to_wrist_flange" type="fixed">
+      <parent link="world" />
+      <child link="$(arg tf_prefix)robotiq_hande_base_link" />
+      <origin xyz="1 1 0" rpy="0 0 0" />
+    </joint>
    <xacro:if value="$(arg sim_gazebo)">
     <!-- Gazebo plugins -->

Commit message: refactor: code clean up

File: src/ur3e_hande_robot_description/urdf/hande.xacro (robot description, xacro)
@@ -7,8 +7,8 @@
     ur_type
     parent" >
-  <xacro:property name="hande_joint_limit_params" value="$(find ur3e_hande_robot_description)/config/$(arg ur_type)/joint_limits.yaml"/>
-  <xacro:property name="hande_kinematics_params" value="$(find ur3e_hande_robot_description)/config/$(arg ur_type)/default_kinematics.yaml"/>
-  <xacro:property name="hande_physical_params" value="$(find ur3e_hande_robot_description)/config/$(arg ur_type)/physical_parameters.yaml"/>
-  <xacro:property name="hande_visual_params" value="$(find ur3e_hande_robot_description)/config/$(arg ur_type)/visual_parameters.yaml"/>
+  <xacro:property name="hande_joint_limit_params" value="$(find ur3e_hande_robot_description)/config/hande/joint_limits.yaml"/>
+  <xacro:property name="hande_kinematics_params" value="$(find ur3e_hande_robot_description)/config/hande/default_kinematics.yaml"/>
+  <xacro:property name="hande_physical_params" value="$(find ur3e_hande_robot_description)/config/hande/physical_parameters.yaml"/>
+  <xacro:property name="hande_visual_params" value="$(find ur3e_hande_robot_description)/config/hande/visual_parameters.yaml"/>
   <xacro:macro name="cylinder_inertial" params="radius length mass *origin">
     <inertial>
@@ -22,10 +22,5 @@
   <xacro:property name="config_physical_parameters" value="${xacro.load_yaml(hande_physical_params)}"/>
   <!-- Extract subsections from yaml dictionaries -->
-  <!-- <xacro:property name="sec_limits" value="${config_joint_limit_parameters['joint_limits']}"/> -->
-  <!-- <xacro:property name="sec_dh_parameters" value="${config_physical_parameters['dh_parameters']}"/> -->
-  <!-- <xacro:property name="sec_offsets" value="${config_physical_parameters['offsets']}"/> -->
   <xacro:property name="sec_inertia_parameters" value="${config_physical_parameters['inertia_parameters']}" />
-  <!-- <xacro:property name="sec_mesh_files" value="${config_visual_parameters['mesh_files']}" scope="parent"/> -->
-  <!-- <xacro:property name="sec_kinematics" value="${config_kinematics_parameters['kinematics']}" /> -->
   <xacro:property name="intertia_links" value="${sec_inertia_parameters['links']}" scope="parent"/>
   <xacro:property name="hande_base_mass" value="${sec_inertia_parameters['hande_base_mass']}" scope="parent"/>
@@ -44,5 +39,5 @@
   <xacro:property name="hande_base_radius" value="${sec_inertia_parameters['hande_base_radius']}" scope="parent"/>
   <xacro:property name="finger_radius" value="${sec_inertia_parameters['finger_radius']}" scope="parent"/>
-    <!-- customization to include hande -->
+    <!-- customizations to include hande -->
     <link name="${tf_prefix}robotiq_hande_base_link">
       <visual>
@@ -121,9 +116,4 @@
       <mimic joint="${tf_prefix}joint_finger" multiplier="1" offset="0"/>
     </joint>
-    <!-- <joint name="$(arg tf_prefix)hande_to_wrist_flange" type="fixed">
-      <parent link="${parent}" />
-      <child link="${tf_prefix}robotiq_hande_base_link" />
-      <origin xyz="1 1 0" rpy="0 0 0" />
-    </joint> -->
 </xacro:macro>
 </robot>

Commit message: refactor: clean ups

File: src/ur3e_hande_robot_description/urdf/hande.xacro (robot description, xacro)
@@ -5,7 +5,5 @@
     name
     tf_prefix
-    ur_type
     parent" >
-  <xacro:property name="hande_joint_limit_params" value="$(find ur3e_hande_robot_description)/config/hande/joint_limits.yaml"/>
   <xacro:property name="hande_kinematics_params" value="$(find ur3e_hande_robot_description)/config/hande/default_kinematics.yaml"/>
   <xacro:property name="hande_physical_params" value="$(find ur3e_hande_robot_description)/config/hande/physical_parameters.yaml"/>

File: src/ur3e_hande_robot_description/urdf/hande_extension.urdf.xacro (robot description, xacro)
@@ -92,10 +92,11 @@
      <origin xyz="0 0 0" rpy="0 0 0" />          <!-- position robot in the world -->
    </xacro:ur_robot>
+    <!-- Call the robot gripper -->
     <xacro:robotiq_hande
      name="$(arg name)"
      tf_prefix="$(arg tf_prefix)"
-     ur_type="$(arg ur_type)"
      parent="world"
    />
+    <!-- attach the gripper to the arm -->
     <joint name="$(arg tf_prefix)hande_to_wrist_flange" type="fixed">
       <parent link="$(arg tf_prefix)flange" />

Commit message: fix: urdf hande joints

File: src/ur3e_hande_robot_description/urdf/hande.xacro (robot description, xacro)
@@ -100,5 +100,5 @@
     </link>
     <!-- hande installation -->
-    <joint name="${tf_prefix}joint_finger" type="prismatic">
+    <joint name="${tf_prefix}joint_finger" type="fixed">
       <origin rpy="0 0 0" xyz="0 0 0.099"/>
       <parent link="${tf_prefix}robotiq_hande_base_link"/>
@@ -107,5 +107,5 @@
       <limit effort="130" lower="0" upper="0.025" velocity="0.15"/>
     </joint>
-    <joint name="robotiq_hande_base_to_${tf_prefix}right_finger" type="prismatic">
+    <joint name="robotiq_hande_base_to_${tf_prefix}right_finger" type="fixed">
       <origin rpy="0 0 0" xyz="0 0 0.099"/>
       <parent link="${tf_prefix}robotiq_hande_base_link"/>

Commit message: feat: add a grasping point

File: src/ur3e_hande_robot_description/urdf/hande.xacro (robot description, xacro)
@@ -99,4 +99,9 @@
       </xacro:cylinder_inertial>
     </link>
+    <link name="grasping_point_link">
+      <visual>
+        <origin rpy="0 0 0" xyz="0 0 0"/>
+       </visual>
+    </link>
     <!-- hande installation -->
     <joint name="${tf_prefix}joint_finger" type="fixed">
@@ -115,4 +120,10 @@
       <mimic joint="${tf_prefix}joint_finger" multiplier="1" offset="0"/>
     </joint>
+    <joint name="${tf_prefix}grasping_point" type="fixed">
+      <origin rpy="0 0 0" xyz="0.1 0.2 0.099"/>
+      <parent link="${tf_prefix}robotiq_hande_base_link"/>
+      <child link="grasping_point_link"/>
+      <axis xyz="-1 0 0"/>
+    </joint>
 </xacro:macro>
 </robot>

Commit message: fix: gripper point coords

File: src/ur3e_hande_robot_description/urdf/hande.xacro (robot description, xacro)
@@ -121,8 +121,8 @@
     </joint>
     <joint name="${tf_prefix}grasping_point" type="fixed">
-      <origin rpy="0 0 0" xyz="0.1 0.2 0.099"/>
+      <origin rpy="0 0 0" xyz="0.0 0.0 0.134"/>
       <parent link="${tf_prefix}robotiq_hande_base_link"/>
       <child link="grasping_point_link"/>
-      <axis xyz="-1 0 0"/>
+      <axis xyz="0 0 0"/>
     </joint>
 </xacro:macro>

Commit message: fix: move the grasping point

File: src/ur3e_hande_robot_description/urdf/hande.xacro (robot description, xacro)
@@ -39,4 +39,5 @@
   <xacro:property name="finger_radius" value="${sec_inertia_parameters['finger_radius']}" scope="parent"/>
     <!-- customizations to include hande -->
+    <!-- TODO: Add the coupler between the wrist_3_link and robotiq_hande_base_link -->
     <link name="${tf_prefix}robotiq_hande_base_link">
       <visual>
@@ -100,7 +101,4 @@
     </link>
     <link name="grasping_point_link">
-      <visual>
-        <origin rpy="0 0 0" xyz="0 0 0"/>
-       </visual>
     </link>
     <!-- hande installation -->
@@ -121,5 +119,5 @@
     </joint>
     <joint name="${tf_prefix}grasping_point" type="fixed">
-      <origin rpy="0 0 0" xyz="0.0 0.0 0.134"/>
+      <origin rpy="0 0 0" xyz="0.0 0.0 0.15"/>
       <parent link="${tf_prefix}robotiq_hande_base_link"/>
       <child link="grasping_point_link"/>

Commit message: fix: add visual for grasp point

File: src/ur3e_hande_robot_description/urdf/hande.xacro (robot description, xacro)
@@ -101,4 +101,7 @@
     </link>
     <link name="grasping_point_link">
+        <visual>
+          <origin rpy="0 0 0" xyz="0 0 0"/>
+       </visual>
     </link>
     <!-- hande installation -->

Commit message: fix: grasping point

File: src/ur3e_hande_robot_description/urdf/hande.xacro (robot description, xacro)
@@ -122,5 +122,5 @@
     </joint>
     <joint name="${tf_prefix}grasping_point" type="fixed">
-      <origin rpy="0 0 0" xyz="0.0 0.0 0.15"/>
+      <origin rpy="0 0 0" xyz="0.0 0.0 0.16"/>
       <parent link="${tf_prefix}robotiq_hande_base_link"/>
       <child link="grasping_point_link"/>

Commit message: fix: gripper point

File: src/ur3e_hande_robot_description/urdf/hande.xacro (robot description, xacro)
@@ -122,5 +122,5 @@
     </joint>
     <joint name="${tf_prefix}grasping_point" type="fixed">
-      <origin rpy="0 0 0" xyz="0.0 0.0 0.16"/>
+      <origin rpy="0 0 0" xyz="0.0 0.0 0.15"/>
       <parent link="${tf_prefix}robotiq_hande_base_link"/>
       <child link="grasping_point_link"/>

Commit message: fix: gripper point

File: src/ur3e_hande_robot_description/urdf/hande.xacro (robot description, xacro)
@@ -101,7 +101,7 @@
     </link>
     <link name="grasping_point_link">
-        <visual>
-          <origin rpy="0 0 0" xyz="0 0 0"/>
-       </visual>
+      <visual>
+        <origin rpy="0 0 0" xyz="0 0 0"/>
+      </visual>
     </link>
     <!-- hande installation -->

Commit message: fix: gripper tests

File: src/ur3e_hande_robot_description/urdf/hande.xacro (robot description, xacro)
@@ -122,5 +122,5 @@
     </joint>
     <joint name="${tf_prefix}grasping_point" type="fixed">
-      <origin rpy="0 0 0" xyz="0.0 0.0 0.15"/>
+      <origin rpy="0 0 0" xyz="0.0 0.0 0.135"/>
       <parent link="${tf_prefix}robotiq_hande_base_link"/>
       <child link="grasping_point_link"/>

Commit message: fix: hande xacro from old

File: src/ur3e_hande_robot_description/urdf/hande.xacro (robot description, xacro)
@@ -103,5 +103,5 @@
       <visual>
         <origin rpy="0 0 0" xyz="0 0 0"/>
-      </visual>
+       </visual>
     </link>
     <!-- hande installation -->
@@ -122,5 +122,5 @@
     </joint>
     <joint name="${tf_prefix}grasping_point" type="fixed">
-      <origin rpy="0 0 0" xyz="0.0 0.0 0.135"/>
+      <origin rpy="0 0 0" xyz="0.0 0.0 0.15"/>
       <parent link="${tf_prefix}robotiq_hande_base_link"/>
       <child link="grasping_point_link"/>

Commit message: fix: remove visual for grasp point

File: src/ur3e_hande_robot_description/urdf/hande.xacro (robot description, xacro)
@@ -100,7 +100,4 @@
     </link>
     <link name="grasping_point_link">
-      <visual>
-        <origin rpy="0 0 0" xyz="0 0 0"/>
-       </visual>
     </link>
     <!-- hande installation -->

Commit message: fix: weired error

File: src/ur3e_hande_robot_description/urdf/hande.xacro (robot description, xacro)
@@ -100,4 +100,7 @@
     </link>
     <link name="grasping_point_link">
+      <visual>
+        <origin rpy="0 0 0" xyz="0 0 0"/>
+       </visual>
     </link>
     <!-- hande installation -->

Commit message: fix: use one hande for all + spelling + PR fixes

File: src/ur3e_hande_robot_description/urdf/hande.xacro (robot description, xacro)
@@ -1,13 +1,11 @@
 <?xml version="1.0"?>
-<robot xmlns:xacro="http://wiki.ros.org/xacro" name="$(arg name)">
+<robot xmlns:xacro="http://wiki.ros.org/xacro" name="hande_black">
 <!--Based on same file and version as the https://github.com/AcutronicRobotics/robotiq_modular_gripper/blob/4e708524e5dd20753f711686eb2cd1017a25a09e/robotiq_hande_gripper_description/urdf/robotiq_hande.urdf.xacro-->
-  <xacro:arg name="name" default="hande"/>
 <xacro:macro name="robotiq_hande" params="
-    name
     tf_prefix
     parent" >
   <xacro:property name="hande_kinematics_params" value="$(find ur3e_hande_robot_description)/config/hande/default_kinematics.yaml"/>
   <xacro:property name="hande_physical_params" value="$(find ur3e_hande_robot_description)/config/hande/physical_parameters.yaml"/>
-  <xacro:property name="hande_visual_params" value="$(find ur3e_hande_robot_description)/config/hande/visual_parameters.yaml"/>
+  <!-- <xacro:property name="hande_visual_params" value="$(find ur3e_hande_robot_description)/config/hande/visual_parameters.yaml"/> -->
   <xacro:macro name="cylinder_inertial" params="radius length mass *origin">
     <inertial>
@@ -20,5 +18,4 @@
   </xacro:macro>
   <xacro:property name="config_physical_parameters" value="${xacro.load_yaml(hande_physical_params)}"/>
-  <!-- Extract subsections from yaml dictionaries -->
   <xacro:property name="sec_inertia_parameters" value="${config_physical_parameters['inertia_parameters']}" />
   <xacro:property name="intertia_links" value="${sec_inertia_parameters['links']}" scope="parent"/>
@@ -38,10 +35,33 @@
   <xacro:property name="hande_base_radius" value="${sec_inertia_parameters['hande_base_radius']}" scope="parent"/>
   <xacro:property name="finger_radius" value="${sec_inertia_parameters['finger_radius']}" scope="parent"/>
-    <!-- customizations to include hande -->
+  <xacro:property name="scaling_factor_cp" value="1"/>
+    <link name="${tf_prefix}robotiq_coupler">
+      <inertial>
+        <mass value="0.100" />
+        <inertia
+          ixx="6.17674E-05" ixy="0.0" ixz="0.0"
+          iyy="6.17674E-05" iyz="0.0"
+          izz="1.18125E-04"
+        />
+      </inertial>
+      <collision>
+        <geometry>
+          <mesh filename="package://ur3e_hande_robot_description/meshes/hande/collision/coupler.stl" scale="${scaling_factor_cp} ${scaling_factor_cp} ${scaling_factor_cp}" />
+        </geometry>
+      </collision>
+      <visual>
+        <geometry>
+          <mesh filename="package://ur3e_hande_robot_description/meshes/hande/visual/coupler.dae" scale="${scaling_factor_cp} ${scaling_factor_cp} ${scaling_factor_cp}" />
+        </geometry>
+        <material name="Gazebo/Black">
+          <color rgba="0.1 0.1 0.1 1" />
+        </material>
+      </visual>
+    </link>
     <link name="${tf_prefix}robotiq_hande_base_link">
       <visual>
-        <origin xyz="0 0 0" rpy="0 0 0" />
+        <origin xyz="0 0 0" rpy="0 -1.570796 -1.570796" />
         <geometry>
-          <mesh filename="package://ur3e_hande_robot_description/meshes/hande/visual/hand-e.dae" scale="0.001 0.001 0.001" />
+          <mesh filename="package://ur3e_hande_robot_description/meshes/hande/visual/hande.dae" scale="1 1 1" />
         </geometry>
         <material name="Gazebo/Black">
@@ -50,11 +70,10 @@
       </visual>
       <collision>
-        <origin xyz="0 0 0" rpy="0 0 0" />
         <geometry>
-          <mesh filename="package://ur3e_hande_robot_description/meshes/hande/collision/hand-e.stl" scale="0.001 0.001 0.001"/>
+          <mesh filename="package://ur3e_hande_robot_description/meshes/hande/collision/hande.stl" scale="1 1 1"/>
         </geometry>
       </collision>
       <xacro:cylinder_inertial radius="${hande_base_inertia_radius}" length="${hande_base_inertia_length}"  mass="${hande_base_mass}">
-        <origin xyz="0.0 0.0 ${-0.5 * hande_base_inertia_length}" rpy="0 0 0" />
+        <origin xyz="${hande_base_cog}" rpy="0 0 0" />
       </xacro:cylinder_inertial>
     </link>
@@ -76,5 +95,5 @@
       </collision>
       <xacro:cylinder_inertial radius="${left_finger_inertia_radius}" length="${left_finger_inertia_length}"  mass="${left_finger_mass}">
-        <origin xyz="0.0 0.0 ${-0.5 * left_finger_inertia_length}" rpy="0 0 0" />
+        <origin xyz="${finger_cog}" rpy="0 0 0" />
       </xacro:cylinder_inertial>
     </link>
@@ -96,12 +115,16 @@
       </collision>
       <xacro:cylinder_inertial radius="${right_finger_inertia_radius}" length="${right_finger_inertia_length}"  mass="${right_finger_mass}">
-        <origin xyz="0.0 0.0 ${-0.5 * right_finger_inertia_length}" rpy="0 0 0" />
+        <origin xyz="${finger_cog}" rpy="0 0 0" />
       </xacro:cylinder_inertial>
     </link>
     <link name="grasping_point_link">
     </link>
-    <!-- hande installation -->
+    <joint name="robotiq_coupler_joint" type="fixed">
+      <origin xyz="0 0 -0.05" rpy="${pi} 0 ${-pi/2.0}" />
+      <parent link="${tf_prefix}robotiq_coupler"/>
+      <child link="${tf_prefix}robotiq_hande_base_link"/>
+    </joint>
     <joint name="${tf_prefix}joint_finger" type="fixed">
-      <origin rpy="0 0 0" xyz="0 0 0.099"/>
+      <origin rpy="0 0 ${pi/2.0}" xyz="0 0 0.05"/>
       <parent link="${tf_prefix}robotiq_hande_base_link"/>
       <child link="${tf_prefix}left_finger"/>
@@ -110,5 +133,5 @@
     </joint>
     <joint name="robotiq_hande_base_to_${tf_prefix}right_finger" type="fixed">
-      <origin rpy="0 0 0" xyz="0 0 0.099"/>
+      <origin rpy="0 0 ${pi/2.0}" xyz="0 0 0.05"/>
       <parent link="${tf_prefix}robotiq_hande_base_link"/>
       <child link="${tf_prefix}right_finger"/>
@@ -118,5 +141,5 @@
     </joint>
     <joint name="${tf_prefix}grasping_point" type="fixed">
-      <origin rpy="0 0 0" xyz="0.0 0.0 0.15"/>
+      <origin rpy="0 0 0" xyz="0.0 0.0 0.09"/>
       <parent link="${tf_prefix}robotiq_hande_base_link"/>
       <child link="grasping_point_link"/>

File: src/ur3e_hande_robot_description/urdf/ur_with_camera_hande.xacro (robot description, xacro)
@@ -6,5 +6,5 @@
    <!-- import main macro -->
    <xacro:include filename="$(find ur_description)/urdf/ur_macro.xacro"/>
-  <xacro:include filename="$(find ur3e_hande_robot_description)/urdf/hande_black.xacro"/>
+  <xacro:include filename="$(find ur3e_hande_robot_description)/urdf/hande.xacro"/>
   <xacro:include filename="$(find ur3e_hande_robot_description)/urdf/camera_mount.xacro"/>
    <!-- possible 'ur_type' values: ur3, ur3e, ur5, ur5e, ur10, ur10e, ur16e, ur20 -->

File: src/ur3e_hande_robot_description/urdf/ur_with_hande.xacro (robot description, xacro)
@@ -95,5 +95,4 @@
     <!-- Call the robot gripper -->
     <xacro:robotiq_hande
-     name="$(arg name)"
      tf_prefix="$(arg tf_prefix)"
      parent="world"
@@ -102,6 +101,7 @@
     <joint name="$(arg tf_prefix)hande_to_wrist_flange" type="fixed">
       <parent link="$(arg tf_prefix)flange" />
-      <child link="$(arg tf_prefix)robotiq_hande_base_link" />
-      <origin xyz="0 0 0" rpy="${pi/2.0} 0 ${pi/2.0}" />
+      <!-- <child link="$(arg tf_prefix)robotiq_hande_base_link" /> -->
+      <child link="$(arg tf_prefix)robotiq_coupler" />
+      <origin xyz="0.005 0 0" rpy="-${pi/2.0} 0 ${pi/2.0}" />
     </joint>
 </robot>
