Commit message: fix: correct xacros

File: src/ur3e_hande_robot_description/urdf/camera_mount.xacro (robot description, xacro)
@@ -6,4 +6,5 @@
   <!-- Mass and Inertial properties -->
   <xacro:property name="mount_mass" value="${mount_physical_parameters['inertia_parameters']['mount_base_mass']}"/> <!-- Mass in kg -->
+  <xacro:property name="camera_mass" value="${mount_physical_parameters['inertia_parameters']['camera_mass']}"/> <!-- Mass in kg -->
   <!-- <xacro:property name="intertia_links" value="${mount_physical_parameters['links']}" scope="parent"/> -->
   <!-- Dimensions of the rectangular object -->
@@ -11,4 +12,8 @@
   <xacro:property name="mount_width" value="${mount_physical_parameters['inertia_parameters']['links']['mount_base']['width']}" scope="parent"/>   <!-- Width in meters -->
   <xacro:property name="mount_height" value="${mount_physical_parameters['inertia_parameters']['links']['mount_base']['height']}" scope="parent"/>  <!-- Height in meters -->
+  <!-- Dimensions of the camera -->
+  <xacro:property name="camera_length" value="${mount_physical_parameters['inertia_parameters']['links']['camera']['length']}" scope="parent"/>  <!-- Length in meters -->
+  <xacro:property name="camera_width" value="${mount_physical_parameters['inertia_parameters']['links']['camera']['width']}" scope="parent"/>   <!-- Width in meters -->
+  <xacro:property name="camera_height" value="${mount_physical_parameters['inertia_parameters']['links']['camera']['height']}" scope="parent"/>  <!-- Height in meters -->
   <xacro:property name="scaling_factor" value="0.0265"/>
   <xacro:macro name="rectangular_inertial" params="length width height mass *origin">
@@ -42,4 +47,29 @@
     </xacro:rectangular_inertial>
   </link>
+  <xacro:property name="scaling_factor_cm" value="0.0009"/>
+  <link name="camera_base">
+    <visual>
+      <!-- <origin xyz="-0.013 0. 0." /> -->
+        <geometry>
+          <mesh filename="package://ur3e_hande_robot_description/meshes/camera_mount/visual/azure_kinect.dae" scale="${scaling_factor_cm} ${scaling_factor_cm} ${scaling_factor_cm}" />
+        </geometry>
+        <material name="Gazebo/Black">
+          <color rgba="0.1 0.1 0.1 1" />
+        </material>
+    </visual>
+    <collision>
+      <geometry>
+        <mesh filename="package://ur3e_hande_robot_description/meshes/camera_mount/collision/azure_kinect.stl" scale="${scaling_factor_cm} ${scaling_factor_cm} ${scaling_factor_cm}" />
+      </geometry>
+    </collision>
+    <xacro:rectangular_inertial length="${camera_length}"  width="${camera_width}"  height="${camera_height}" mass="${camera_mass}">
+        <origin xyz="0.0 0.0 0.0" rpy="0 0 0" />
+    </xacro:rectangular_inertial>
+  </link>
+   <joint name="camera_base_to_mount" type="fixed">
+    <parent link="mount" />
+    <child link="camera_base" />
+    <origin xyz="0. -0.055 0.0725" rpy="${pi/2} 0. 0." />
+  </joint>
   </xacro:macro>
 </robot>

File: src/ur3e_hande_robot_description/urdf/hande_black.xacro (robot description, xacro)
@@ -1,8 +1,6 @@
 <?xml version="1.0"?>
-<robot xmlns:xacro="http://wiki.ros.org/xacro" name="$(arg name)">
+<robot xmlns:xacro="http://wiki.ros.org/xacro" name="hande_black">
 <!--Based on same file and version as the https://github.com/AcutronicRobotics/robotiq_modular_gripper/blob/4e708524e5dd20753f711686eb2cd1017a25a09e/robotiq_hande_gripper_description/urdf/robotiq_hande.urdf.xacro-->
-  <xacro:arg name="name" default="hande"/>
 <xacro:macro name="robotiq_hande" params="
-    name
     tf_prefix
     parent" >
@@ -122,4 +120,9 @@
     <link name="grasping_point_link">
     </link>
+    <joint name="robotiq_coupler_joint" type="fixed">
+      <origin xyz="0 0 -0.05" rpy="${pi} 0 ${-pi/2.0}" />
+      <parent link="${tf_prefix}robotiq_coupler"/>
+      <child link="${tf_prefix}robotiq_hande_base_link"/>
+    </joint>
     <joint name="${tf_prefix}joint_finger" type="fixed">
       <origin rpy="0 0 ${pi/2.0}" xyz="0 0 0.05"/>
@@ -143,9 +146,4 @@
       <axis xyz="0 0 0"/>
     </joint>
-    <joint name="robotiq_coupler_joint" type="fixed">
-      <origin xyz="0 0 -0.05" rpy="${pi} 0 ${-pi/2.0}" />
-      <parent link="${tf_prefix}robotiq_coupler"/>
-      <child link="${tf_prefix}robotiq_hande_base_link"/>
-    </joint>
 </xacro:macro>
 </robot>

Commit message: feat: new dae wip aruco

File: src/ur3e_hande_robot_description/urdf/camera_mount.xacro (robot description, xacro)
@@ -70,5 +70,5 @@
     <parent link="mount" />
     <child link="camera_base" />
-    <origin xyz="0. -0.055 0.0725" rpy="${pi/2} 0. 0." />
+    <origin xyz="0. -0.09 0.0725" rpy="${pi/2} 0. 0." />
   </joint>
   </xacro:macro>

Commit message: feat: add visor tf

File: src/ur3e_hande_robot_description/urdf/camera_mount.xacro (robot description, xacro)
@@ -67,9 +67,16 @@
     </xacro:rectangular_inertial>
   </link>
-   <joint name="camera_base_to_mount" type="fixed">
+  <link name="camera_base_map">
+  </link>
+  <joint name="camera_base_to_mount" type="fixed">
     <parent link="mount" />
     <child link="camera_base" />
     <origin xyz="0. -0.09 0.0725" rpy="${pi/2} 0. 0." />
   </joint>
+  <joint name="camera_base_to_camera_base_map" type="fixed">
+    <parent link="camera_base" />
+    <child link="camera_base_map" />
+    <origin xyz="0. 0.0 0.0315" rpy="${pi/2} 0. 0." />
+  </joint>
   </xacro:macro>
 </robot>

Commit message: fix: correct cog

File: src/ur3e_hande_robot_description/urdf/camera_mount.xacro (robot description, xacro)
@@ -4,4 +4,5 @@
   <xacro:property name="mount_physical_params_file" value="$(find ur3e_hande_robot_description)/config/camera_mount/physical_parameters.yaml"/>
   <xacro:property name="mount_physical_parameters" value="${xacro.load_yaml(mount_physical_params_file)}"/>
+  <!-- <xacro:property name="sec_inertia_parameters" value="${mount_physical_parameters['inertia_parameters']}" /> -->
   <!-- Mass and Inertial properties -->
   <xacro:property name="mount_mass" value="${mount_physical_parameters['inertia_parameters']['mount_base_mass']}"/> <!-- Mass in kg -->
@@ -16,4 +17,8 @@
   <xacro:property name="camera_width" value="${mount_physical_parameters['inertia_parameters']['links']['camera']['width']}" scope="parent"/>   <!-- Width in meters -->
   <xacro:property name="camera_height" value="${mount_physical_parameters['inertia_parameters']['links']['camera']['height']}" scope="parent"/>  <!-- Height in meters -->
+  <xacro:property name="prep_mount_cog" value="${mount_physical_parameters['inertia_parameters']['center_of_mass']['mount_cog']}" scope="parent"/>
+  <xacro:property name="cam_cog" value="${mount_physical_parameters['inertia_parameters']['center_of_mass']['camera_cog']}" scope="parent"/>
+  <xacro:property name="mount_cog" value="${prep_mount_cog['x']} ${prep_mount_cog['y']} ${prep_mount_cog['z']}" scope="parent"/>
+  <xacro:property name="camera_cog" value="${cam_cog['x']} ${cam_cog['y']} ${cam_cog['z']}" scope="parent"/>
   <xacro:property name="scaling_factor" value="0.0265"/>
   <xacro:macro name="rectangular_inertial" params="length width height mass *origin">
@@ -44,5 +49,5 @@
     </collision>
     <xacro:rectangular_inertial length="${mount_length}"  width="${mount_width}"  height="${mount_height}" mass="${mount_mass}">
-        <origin xyz="0.0 0.0 0.0" rpy="0 0 0" />
+        <origin xyz="${mount_cog}" rpy="0 0 0" />
     </xacro:rectangular_inertial>
   </link>
@@ -64,5 +69,5 @@
     </collision>
     <xacro:rectangular_inertial length="${camera_length}"  width="${camera_width}"  height="${camera_height}" mass="${camera_mass}">
-        <origin xyz="0.0 0.0 0.0" rpy="0 0 0" />
+        <origin xyz="${camera_cog}" rpy="0 0 0" />
     </xacro:rectangular_inertial>
   </link>

File: src/ur3e_hande_robot_description/urdf/hande_black.xacro (robot description, xacro)
@@ -74,13 +74,6 @@
         </geometry>
       </collision>
-            <!-- <inertial>
-        <inertial
-            ixx="0.005341" ixy="0.0" ixz="0.0"
-            iyy="0.005447" iyz="0.0"
-            izz="0.000636"
-        />
-      </inertial> -->
       <xacro:cylinder_inertial radius="${hande_base_inertia_radius}" length="${hande_base_inertia_length}"  mass="${hande_base_mass}">
-        <origin xyz="0.0 0.0 ${-0.5 * hande_base_inertia_length}" rpy="0 0 0" />
+        <origin xyz="${hande_base_cog}" rpy="0 0 0" />
       </xacro:cylinder_inertial>
     </link>
@@ -102,5 +95,5 @@
       </collision>
       <xacro:cylinder_inertial radius="${left_finger_inertia_radius}" length="${left_finger_inertia_length}"  mass="${left_finger_mass}">
-        <origin xyz="0.0 0.0 ${-0.5 * left_finger_inertia_length}" rpy="0 0 0" />
+        <origin xyz="${finger_cog}" rpy="0 0 0" />
       </xacro:cylinder_inertial>
     </link>
@@ -122,5 +115,5 @@
       </collision>
       <xacro:cylinder_inertial radius="${right_finger_inertia_radius}" length="${right_finger_inertia_length}"  mass="${right_finger_mass}">
-        <origin xyz="0.0 0.0 ${-0.5 * right_finger_inertia_length}" rpy="0 0 0" />
+        <origin xyz="${finger_cog}" rpy="0 0 0" />
       </xacro:cylinder_inertial>
     </link>

Commit message: refac: clean up code

File: src/ur3e_hande_robot_description/urdf/camera_mount.xacro (robot description, xacro)
@@ -4,5 +4,4 @@
   <xacro:property name="mount_physical_params_file" value="$(find ur3e_hande_robot_description)/config/camera_mount/physical_parameters.yaml"/>
   <xacro:property name="mount_physical_parameters" value="${xacro.load_yaml(mount_physical_params_file)}"/>
-  <!-- <xacro:property name="sec_inertia_parameters" value="${mount_physical_parameters['inertia_parameters']}" /> -->
   <!-- Mass and Inertial properties -->
   <xacro:property name="mount_mass" value="${mount_physical_parameters['inertia_parameters']['mount_base_mass']}"/> <!-- Mass in kg -->
@@ -55,5 +54,4 @@
   <link name="camera_base">
     <visual>
-      <!-- <origin xyz="-0.013 0. 0." /> -->
         <geometry>
           <mesh filename="package://ur3e_hande_robot_description/meshes/camera_mount/visual/azure_kinect.dae" scale="${scaling_factor_cm} ${scaling_factor_cm} ${scaling_factor_cm}" />

Commit message: refac: remove comments

File: src/ur3e_hande_robot_description/urdf/camera_mount.xacro (robot description, xacro)
@@ -7,5 +7,4 @@
   <xacro:property name="mount_mass" value="${mount_physical_parameters['inertia_parameters']['mount_base_mass']}"/> <!-- Mass in kg -->
   <xacro:property name="camera_mass" value="${mount_physical_parameters['inertia_parameters']['camera_mass']}"/> <!-- Mass in kg -->
-  <!-- <xacro:property name="intertia_links" value="${mount_physical_parameters['links']}" scope="parent"/> -->
   <!-- Dimensions of the rectangular object -->
   <xacro:property name="mount_length" value="${mount_physical_parameters['inertia_parameters']['links']['mount_base']['length']}" scope="parent"/>  <!-- Length in meters -->

File: src/ur3e_hande_robot_description/urdf/hande.xacro (robot description, xacro)
@@ -7,5 +7,4 @@
   <xacro:property name="hande_kinematics_params" value="$(find ur3e_hande_robot_description)/config/hande/default_kinematics.yaml"/>
   <xacro:property name="hande_physical_params" value="$(find ur3e_hande_robot_description)/config/hande/physical_parameters.yaml"/>
-  <!-- <xacro:property name="hande_visual_params" value="$(find ur3e_hande_robot_description)/config/hande/visual_parameters.yaml"/> -->
   <xacro:macro name="cylinder_inertial" params="radius length mass *origin">
     <inertial>

File: src/ur3e_hande_robot_description/urdf/ur_with_hande.xacro (robot description, xacro)
@@ -101,5 +101,4 @@
     <joint name="$(arg tf_prefix)hande_to_wrist_flange" type="fixed">
       <parent link="$(arg tf_prefix)flange" />
-      <!-- <child link="$(arg tf_prefix)robotiq_hande_base_link" /> -->
       <child link="$(arg tf_prefix)robotiq_coupler" />
       <origin xyz="0.005 0 0" rpy="-${pi/2.0} 0 ${pi/2.0}" />
